File: PCB/guilty-pad-xx-accent-core-plus-yuri.kicad_pcb (KiCad board)
At the start: 2 copper layers, 347.9 x 125.8 mm, 279 parts, among them J1 Conn_01x04_Socket, Q1 G1NP02ELL, SW1 SW_Push, SW10 SW_Push, SW11 SW_Push, SW12 SW_Push, SW13 SW_Push, SW14 SW_Push, SW15 SW_Push, SW16 SW_Push, SW17 SW_Push, SW18 SW_Push, SW19 SW_Push, SW2 SW_Push, SW20 SW_Push, SW21 SW_Push, SW22 SW_Push, SW23 SW_Push, SW24 SW_Push, SW25 SW_Push, SW26 SW_Push, SW27 SW_Push, SW28 SW_Push, SW29 SW_Push, SW3 SW_Push, SW30 SW_Push, SW31 SW_Push, SW32 SW_Push, SW33 SW_Push, SW34 SW_Push, SW35 SW_Push, SW36 SW_Push, SW37 SW_Push, SW38 SW_Push, SW39 SW_Push, SW4 SW_Push, SW40 SW_Push, SW41 SW_Push, SW42 SW_Push, SW43 SW_Push, SW44 SW_Push, SW45 SW_Push, SW46 SW_Push, SW47 SW_Push, SW48 SW_Push, SW49 SW_Push, SW5 SW_Push, SW50 SW_Push, SW51 SW_Push, SW52 SW_Push, SW53 SW_Push, SW54 SW_Push, SW55 SW_Push, SW56 SW_Push, SW57 SW_Push, SW58 SW_Push, SW59 SW_Push, SW6 SW_Push, SW60 SW_Push, SW61 SW_Push, SW62 SW_Push, SW63 SW_Push, SW64 SW_Push, SW65 SW_Push, SW66 SW_Push, SW67 SW_Push, SW68 SW_Push, SW69 SW_Push, SW7 SW_Push, SW70 SW_Push, SW71 SW_Push, SW72 SW_Push, SW73 SW_Push, SW74 SW_Push, SW75 SW_Push, SW76 SW_Push, SW77 SW_Push, SW78 SW_Push, SW79 SW_Push, SW8 SW_Push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

Commit message: idkkkkkkk
Parts:
- added D88: D, Diode_SMD:D_SOD-323_HandSoldering, F.Cu at (76.5, 49.5)
- added G***: LOGO, LOGO, B.Cu at (184.1, 139.8)
- added Q1: Q_PMOS, Package_TO_SOT_SMD:SOT-23_Handsoldering, F.Cu at (66.7, 52.4)
- added Q3: Q_PMOS, Package_TO_SOT_SMD:SOT-23_Handsoldering, F.Cu at (70.7, 55.3)
- added R5: 4.7kΩ, Capacitor_SMD:C_0402_1005Metric_Pad0.74x0.62mm_HandSolder, F.Cu at (147.6, 47.6)
- added REF**: STAB_MX_2.25u, marbastlib-mx:STAB_MX_2.25u, F.Cu at (292.9, 104.8)
- added REF**: STAB_MX_6.25u, marbastlib-mx:STAB_MX_6.25u, F.Cu at (159.5, 142.9)
- added REF**: STAB_MX_2.75u, marbastlib-mx:STAB_MX_2.75u, F.Cu at (288.1, 123.8)
- added REF**: STAB_MX_2.25u, marbastlib-mx:STAB_MX_2.25u, F.Cu at (50.0, 123.8)
- added REF**: STAB_MX_2u, marbastlib-mx:STAB_MX_2u, F.Cu at (295.3, 66.7)
- added TP3: TestPoint, TestPoint:TestPoint_Pad_D1.5mm, B.Cu at (42.4, 57.4)
- added TP4: TestPoint, TestPoint:TestPoint_Pad_D1.5mm, B.Cu at (39.4, 54.2)
- added U5: 74LV1T08GW, Package_TO_SOT_SMD:SOT-353_SC-70-5, F.Cu at (76.0, 53.0)
- D1: renamed from D88; footprint Diode_SMD:D_SMA_Handsoldering -> Diode_SMD:D_SOD-323_HandSoldering; moved to F.Cu
- D10, D11, D12, D13, D14, D15, D16, D17, D18, D19, D2, D20, D21, D22, D23, D24, D25, D26, D27, D28, D29, D3, D30, D31, D32, D33, D34, D35, D36, D37, D38, D39, D4, D40, D41, D42, D43, D44, D45, D46, D47, D48, D49, D5, D50, D51, D52, D53, D54, D55, D56, D57, D58, D59, D6, D60, D61, D62, D63, D64, D65, D66, D67, D68, D69, D7, D70, D71, D72, D73, D74, D75, D76, D77, D78, D79, D8, D80, D81, D82, D83, D84, D85, D86, D87, D9: footprint Diode_SMD:D_SMA_Handsoldering -> Diode_SMD:D_SOD-323_HandSoldering; moved to F.Cu
- D88: renamed from D1; footprint Diode_SMD:D_SMA_Handsoldering -> Diode_SMD:D_SOD-323_HandSoldering
- D89: footprint Diode_SMD:D_SMA_Handsoldering -> Diode_SMD:D_SOD-323_HandSoldering
- LED1, LED10, LED11, LED12, LED13, LED14, LED15, LED16, LED17, LED18, LED19, LED2, LED20, LED21, LED22, LED23, LED24, LED25, LED26, LED27, LED28, LED29, LED3, LED30, LED31, LED32, LED33, LED34, LED35, LED36, LED37, LED38, LED39, LED4, LED40, LED41, LED42, LED43, LED44, LED45, LED46, LED47, LED48, LED49, LED5, LED50, LED51, LED52, LED53, LED54, LED55, LED56, LED57, LED58, LED59, LED6, LED60, LED61, LED62, LED63, LED64, LED65, LED66, LED67, LED68, LED69, LED7, LED70, LED71, LED72, LED73, LED74, LED75, LED76, LED77, LED78, LED79, LED8, LED80, LED81, LED82, LED83, LED84, LED85, LED86, LED87, LED9: value MX_SK6803MINI-E -> SK6803MINI-E
- SW1: renamed from SW87; footprint gpxxacpy:SW_Cherry_MX_1.00u_PCB -> marbastlib-mx:SW_MX_HS_CPG151101S11_1u; moved to B.Cu
- SW10: renamed from SW9; footprint gpxxacpy:SW_Cherry_MX_1.00u_PCB -> marbastlib-mx:SW_MX_HS_CPG151101S11_1u; moved to B.Cu
- SW11: renamed from SW10; footprint gpxxacpy:SW_Cherry_MX_1.00u_PCB -> marbastlib-mx:SW_MX_HS_CPG151101S11_1u; moved to B.Cu
- SW12: renamed from SW11; footprint gpxxacpy:SW_Cherry_MX_1.00u_PCB -> marbastlib-mx:SW_MX_HS_CPG151101S11_1u; moved to B.Cu
- SW13: renamed from SW12; footprint gpxxacpy:SW_Cherry_MX_1.00u_PCB -> marbastlib-mx:SW_MX_HS_CPG151101S11_1u; moved to B.Cu
- SW14: renamed from SW13; footprint gpxxacpy:SW_Cherry_MX_1.00u_PCB -> marbastlib-mx:SW_MX_HS_CPG151101S11_1u; moved to B.Cu
- SW15: renamed from SW14; footprint gpxxacpy:SW_Cherry_MX_1.00u_PCB -> marbastlib-mx:SW_MX_HS_CPG151101S11_1u; moved to B.Cu
- SW16: renamed from SW15; footprint gpxxacpy:SW_Cherry_MX_1.00u_PCB -> marbastlib-mx:SW_MX_HS_CPG151101S11_1u; moved to B.Cu
- SW17: renamed from SW16; footprint gpxxacpy:SW_Cherry_MX_1.00u_PCB -> marbastlib-mx:SW_MX_HS_CPG151101S11_1u; moved to B.Cu
- SW18: renamed from SW17; footprint gpxxacpy:SW_Cherry_MX_1.00u_PCB -> marbastlib-mx:SW_MX_HS_CPG151101S11_1u; moved to B.Cu
- SW19: renamed from SW18; footprint gpxxacpy:SW_Cherry_MX_1.00u_PCB -> marbastlib-mx:SW_MX_HS_CPG151101S11_1u; moved to B.Cu
- SW2: renamed from SW1; footprint gpxxacpy:SW_Cherry_MX_1.00u_PCB -> marbastlib-mx:SW_MX_HS_CPG151101S11_1u; moved to B.Cu
- SW20: renamed from SW19; footprint gpxxacpy:SW_Cherry_MX_1.00u_PCB -> marbastlib-mx:SW_MX_HS_CPG151101S11_1u; moved to B.Cu
- SW21: renamed from SW20; footprint gpxxacpy:SW_Cherry_MX_1.00u_PCB -> marbastlib-mx:SW_MX_HS_CPG151101S11_1u; moved to B.Cu
- SW22: renamed from SW21; footprint gpxxacpy:SW_Cherry_MX_1.00u_PCB -> marbastlib-mx:SW_MX_HS_CPG151101S11_1u; moved to B.Cu
- SW23: renamed from SW22; footprint gpxxacpy:SW_Cherry_MX_1.00u_PCB -> marbastlib-mx:SW_MX_HS_CPG151101S11_1u; moved to B.Cu
- SW24: renamed from SW23; footprint gpxxacpy:SW_Cherry_MX_1.00u_PCB -> marbastlib-mx:SW_MX_HS_CPG151101S11_1u; moved to B.Cu
- SW25: renamed from SW24; footprint gpxxacpy:SW_Cherry_MX_1.00u_PCB -> marbastlib-mx:SW_MX_HS_CPG151101S11_1u; moved to B.Cu
- SW26: renamed from SW25; footprint gpxxacpy:SW_Cherry_MX_1.00u_PCB -> marbastlib-mx:SW_MX_HS_CPG151101S11_1u; moved to B.Cu
- SW27: renamed from SW26; footprint gpxxacpy:SW_Cherry_MX_1.00u_PCB -> marbastlib-mx:SW_MX_HS_CPG151101S11_1u; moved to B.Cu
- SW28: renamed from SW27; footprint gpxxacpy:SW_Cherry_MX_1.00u_PCB -> marbastlib-mx:SW_MX_HS_CPG151101S11_1u; moved to B.Cu
- SW29: renamed from SW28; footprint gpxxacpy:SW_Cherry_MX_1.00u_PCB -> marbastlib-mx:SW_MX_HS_CPG151101S11_1u; moved to B.Cu
- SW3: renamed from SW2; footprint gpxxacpy:SW_Cherry_MX_1.00u_PCB -> marbastlib-mx:SW_MX_HS_CPG151101S11_1u; moved to B.Cu
- SW30: renamed from SW29; footprint gpxxacpy:SW_Cherry_MX_2.00u_PCB -> marbastlib-mx:SW_MX_HS_CPG151101S11_1u; moved to B.Cu
- SW31: renamed from SW30; footprint gpxxacpy:SW_Cherry_MX_1.00u_PCB -> marbastlib-mx:SW_MX_HS_CPG151101S11_1u; moved to B.Cu
- SW32: renamed from SW31; footprint gpxxacpy:SW_Cherry_MX_1.00u_PCB -> marbastlib-mx:SW_MX_HS_CPG151101S11_1u; moved to B.Cu
- SW33: renamed from SW32; footprint gpxxacpy:SW_Cherry_MX_1.00u_PCB -> marbastlib-mx:SW_MX_HS_CPG151101S11_1u; moved to B.Cu
- SW34: renamed from SW33; footprint gpxxacpy:SW_Cherry_MX_1.00u_PCB -> marbastlib-mx:SW_MX_HS_CPG151101S11_1u; moved to B.Cu
- SW35: renamed from SW34; footprint gpxxacpy:SW_Cherry_MX_1.50u_PCB -> marbastlib-mx:SW_MX_HS_CPG151101S11_1.5u; moved to B.Cu
- SW36: renamed from SW35; footprint gpxxacpy:SW_Cherry_MX_1.00u_PCB -> marbastlib-mx:SW_MX_HS_CPG151101S11_1u; moved to B.Cu
- SW37: renamed from SW36; footprint gpxxacpy:SW_Cherry_MX_1.00u_PCB -> marbastlib-mx:SW_MX_HS_CPG151101S11_1u; moved to B.Cu
- SW38: renamed from SW37; footprint gpxxacpy:SW_Cherry_MX_1.00u_PCB -> marbastlib-mx:SW_MX_HS_CPG151101S11_1u; moved to B.Cu
- SW39: renamed from SW38; footprint gpxxacpy:SW_Cherry_MX_1.00u_PCB -> marbastlib-mx:SW_MX_HS_CPG151101S11_1u; moved to B.Cu
- SW4: renamed from SW3; footprint gpxxacpy:SW_Cherry_MX_1.00u_PCB -> marbastlib-mx:SW_MX_HS_CPG151101S11_1u; moved to B.Cu
- SW40: renamed from SW39; footprint gpxxacpy:SW_Cherry_MX_1.00u_PCB -> marbastlib-mx:SW_MX_HS_CPG151101S11_1u; moved to B.Cu
- SW41: renamed from SW40; footprint gpxxacpy:SW_Cherry_MX_1.00u_PCB -> marbastlib-mx:SW_MX_HS_CPG151101S11_1u; moved to B.Cu
- SW42: renamed from SW41; footprint gpxxacpy:SW_Cherry_MX_1.00u_PCB -> marbastlib-mx:SW_MX_HS_CPG151101S11_1u; moved to B.Cu
- SW43: renamed from SW42; footprint gpxxacpy:SW_Cherry_MX_1.00u_PCB -> marbastlib-mx:SW_MX_HS_CPG151101S11_1u; moved to B.Cu
- SW44: renamed from SW43; footprint gpxxacpy:SW_Cherry_MX_1.00u_PCB -> marbastlib-mx:SW_MX_HS_CPG151101S11_1u; moved to B.Cu
- SW45: renamed from SW44; footprint gpxxacpy:SW_Cherry_MX_1.00u_PCB -> marbastlib-mx:SW_MX_HS_CPG151101S11_1u; moved to B.Cu
- SW46: renamed from SW45; footprint gpxxacpy:SW_Cherry_MX_1.00u_PCB -> marbastlib-mx:SW_MX_HS_CPG151101S11_1u; moved to B.Cu
- SW47: renamed from SW46; footprint gpxxacpy:SW_Cherry_MX_1.00u_PCB -> marbastlib-mx:SW_MX_HS_CPG151101S11_1u; moved to B.Cu
- SW48: renamed from SW47; footprint gpxxacpy:SW_Cherry_MX_1.50u_PCB -> marbastlib-mx:SW_MX_HS_CPG151101S11_1.5u; moved to B.Cu
- SW49: renamed from SW48; footprint gpxxacpy:SW_Cherry_MX_1.00u_PCB -> marbastlib-mx:SW_MX_HS_CPG151101S11_1u; moved to B.Cu
- SW5: renamed from SW4; footprint gpxxacpy:SW_Cherry_MX_1.00u_PCB -> marbastlib-mx:SW_MX_HS_CPG151101S11_1u; moved to B.Cu
- SW50: renamed from SW49; footprint gpxxacpy:SW_Cherry_MX_1.00u_PCB -> marbastlib-mx:SW_MX_HS_CPG151101S11_1u; moved to B.Cu
- SW51: renamed from SW50; footprint gpxxacpy:SW_Cherry_MX_1.00u_PCB -> marbastlib-mx:SW_MX_HS_CPG151101S11_1u; moved to B.Cu
- SW52: renamed from SW51; footprint gpxxacpy:SW_Cherry_MX_1.75u_PCB -> marbastlib-mx:SW_MX_HS_CPG151101S11_1.75u; moved to B.Cu
- SW53: renamed from SW52; footprint gpxxacpy:SW_Cherry_MX_1.00u_PCB -> marbastlib-mx:SW_MX_HS_CPG151101S11_1u; moved to B.Cu
- SW54: renamed from SW53; footprint gpxxacpy:SW_Cherry_MX_1.00u_PCB -> marbastlib-mx:SW_MX_HS_CPG151101S11_1u; moved to B.Cu
- SW55: renamed from SW54; footprint gpxxacpy:SW_Cherry_MX_1.00u_PCB -> marbastlib-mx:SW_MX_HS_CPG151101S11_1u; moved to B.Cu
- SW56: renamed from SW55; footprint gpxxacpy:SW_Cherry_MX_1.00u_PCB -> marbastlib-mx:SW_MX_HS_CPG151101S11_1u; moved to B.Cu
- SW57: renamed from SW56; footprint gpxxacpy:SW_Cherry_MX_1.00u_PCB -> marbastlib-mx:SW_MX_HS_CPG151101S11_1u; moved to B.Cu
- SW58: renamed from SW57; footprint gpxxacpy:SW_Cherry_MX_1.00u_PCB -> marbastlib-mx:SW_MX_HS_CPG151101S11_1u; moved to B.Cu
- SW59: renamed from SW58; footprint gpxxacpy:SW_Cherry_MX_1.00u_PCB -> marbastlib-mx:SW_MX_HS_CPG151101S11_1u; moved to B.Cu
- SW6: renamed from SW5; footprint gpxxacpy:SW_Cherry_MX_1.00u_PCB -> marbastlib-mx:SW_MX_HS_CPG151101S11_1u; moved to B.Cu
- SW60: renamed from SW59; footprint gpxxacpy:SW_Cherry_MX_1.00u_PCB -> marbastlib-mx:SW_MX_HS_CPG151101S11_1u; moved to B.Cu
- SW61: renamed from SW60; footprint gpxxacpy:SW_Cherry_MX_1.00u_PCB -> marbastlib-mx:SW_MX_HS_CPG151101S11_1u; moved to B.Cu
- SW62: renamed from SW61; footprint gpxxacpy:SW_Cherry_MX_1.00u_PCB -> marbastlib-mx:SW_MX_HS_CPG151101S11_1u; moved to B.Cu
- SW63: renamed from SW62; footprint gpxxacpy:SW_Cherry_MX_1.00u_PCB -> marbastlib-mx:SW_MX_HS_CPG151101S11_1u; moved to B.Cu
- SW64: renamed from SW63; footprint gpxxacpy:SW_Cherry_MX_2.25u_PCB -> marbastlib-mx:SW_MX_HS_CPG151101S11_1u; moved to B.Cu
- SW65: renamed from SW64; footprint gpxxacpy:SW_Cherry_MX_2.25u_PCB -> marbastlib-mx:SW_MX_HS_CPG151101S11_1u; moved to B.Cu
- SW66: renamed from SW65; footprint gpxxacpy:SW_Cherry_MX_1.00u_PCB -> marbastlib-mx:SW_MX_HS_CPG151101S11_1u; moved to B.Cu
- SW67: renamed from SW66; footprint gpxxacpy:SW_Cherry_MX_1.00u_PCB -> marbastlib-mx:SW_MX_HS_CPG151101S11_1u; moved to B.Cu
- SW68: renamed from SW67; footprint gpxxacpy:SW_Cherry_MX_1.00u_PCB -> marbastlib-mx:SW_MX_HS_CPG151101S11_1u; moved to B.Cu
- SW69: renamed from SW68; footprint gpxxacpy:SW_Cherry_MX_1.00u_PCB -> marbastlib-mx:SW_MX_HS_CPG151101S11_1u; moved to B.Cu
- SW7: renamed from SW6; footprint gpxxacpy:SW_Cherry_MX_1.00u_PCB -> marbastlib-mx:SW_MX_HS_CPG151101S11_1u; moved to B.Cu
- SW70: renamed from SW69; footprint gpxxacpy:SW_Cherry_MX_1.00u_PCB -> marbastlib-mx:SW_MX_HS_CPG151101S11_1u; moved to B.Cu
- SW71: renamed from SW70; footprint gpxxacpy:SW_Cherry_MX_1.00u_PCB -> marbastlib-mx:SW_MX_HS_CPG151101S11_1u; moved to B.Cu
- SW72: renamed from SW71; footprint gpxxacpy:SW_Cherry_MX_1.00u_PCB -> marbastlib-mx:SW_MX_HS_CPG151101S11_1u; moved to B.Cu
- SW73: renamed from SW72; footprint gpxxacpy:SW_Cherry_MX_1.00u_PCB -> marbastlib-mx:SW_MX_HS_CPG151101S11_1u; moved to B.Cu
- SW74: renamed from SW73; footprint gpxxacpy:SW_Cherry_MX_1.00u_PCB -> marbastlib-mx:SW_MX_HS_CPG151101S11_1u; moved to B.Cu
- SW75: renamed from SW74; footprint gpxxacpy:SW_Cherry_MX_1.00u_PCB -> marbastlib-mx:SW_MX_HS_CPG151101S11_1u; moved to B.Cu
- SW76: renamed from SW75; footprint gpxxacpy:SW_Cherry_MX_2.75u_PCB -> marbastlib-mx:SW_MX_HS_CPG151101S11_1u; moved to B.Cu
- SW77: renamed from SW76; footprint gpxxacpy:SW_Cherry_MX_1.00u_PCB -> marbastlib-mx:SW_MX_HS_CPG151101S11_1u; moved to B.Cu
- SW78: renamed from SW77; footprint gpxxacpy:SW_Cherry_MX_1.25u_PCB -> marbastlib-mx:SW_MX_HS_CPG151101S11_1.25u; moved to B.Cu
- SW79: renamed from SW78; footprint gpxxacpy:SW_Cherry_MX_1.25u_PCB -> marbastlib-mx:SW_MX_HS_CPG151101S11_1.25u; moved to B.Cu
- SW8: renamed from SW7; footprint gpxxacpy:SW_Cherry_MX_1.00u_PCB -> marbastlib-mx:SW_MX_HS_CPG151101S11_1u; moved to B.Cu
- SW80: renamed from SW79; footprint gpxxacpy:SW_Cherry_MX_1.25u_PCB -> marbastlib-mx:SW_MX_HS_CPG151101S11_1.25u; moved to B.Cu
- SW81: renamed from SW80; footprint gpxxacpy:SW_Cherry_MX_6.25u_PCB -> marbastlib-mx:SW_MX_HS_CPG151101S11_1u; moved to B.Cu
- SW82: renamed from SW81; footprint gpxxacpy:SW_Cherry_MX_1.25u_PCB -> marbastlib-mx:SW_MX_HS_CPG151101S11_1.25u; moved to B.Cu
- SW83: renamed from SW82; footprint gpxxacpy:SW_Cherry_MX_1.25u_PCB -> marbastlib-mx:SW_MX_HS_CPG151101S11_1.25u; moved to B.Cu
- SW84: renamed from SW83; footprint gpxxacpy:SW_Cherry_MX_1.25u_PCB -> marbastlib-mx:SW_MX_HS_CPG151101S11_1.25u; moved to B.Cu
- SW85: renamed from SW84; footprint gpxxacpy:SW_Cherry_MX_1.25u_PCB -> marbastlib-mx:SW_MX_HS_CPG151101S11_1.25u; moved to B.Cu
- SW86: renamed from SW85; footprint gpxxacpy:SW_Cherry_MX_1.00u_PCB -> marbastlib-mx:SW_MX_HS_CPG151101S11_1u; moved to B.Cu
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- renumbered SW88 to SW89
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Connections:
- C2 pad 1: /LED_GND -> GND
- L1 pad 1: /VBAT -> Net-(L1-Pad1)
- LED1 pad 1: +5V -> +5V_LED
- LED1 pad 4: /LED_GND -> GND
- LED10 pad 1: +5V -> +5V_LED
- LED10 pad 4: /LED_GND -> GND
- LED11 pad 1: +5V -> +5V_LED
- LED11 pad 4: /LED_GND -> GND
- LED12 pad 1: +5V -> +5V_LED
- LED12 pad 4: /LED_GND -> GND
- LED13 pad 1: +5V -> +5V_LED
- LED13 pad 4: /LED_GND -> GND
- LED14 pad 1: +5V -> +5V_LED
- LED14 pad 4: /LED_GND -> GND
- LED15 pad 1: +5V -> +5V_LED
- LED15 pad 4: /LED_GND -> GND
- LED16 pad 1: +5V -> +5V_LED
- LED16 pad 4: /LED_GND -> GND
- LED17 pad 1: +5V -> +5V_LED
- LED17 pad 4: /LED_GND -> GND
- LED18 pad 1: +5V -> +5V_LED
- LED18 pad 4: /LED_GND -> GND
- LED19 pad 1: +5V -> +5V_LED
- LED19 pad 4: /LED_GND -> GND
- LED2 pad 1: +5V -> +5V_LED
- LED2 pad 4: /LED_GND -> GND
- LED20 pad 1: +5V -> +5V_LED
- LED20 pad 4: /LED_GND -> GND
- LED21 pad 1: +5V -> +5V_LED
- LED21 pad 4: /LED_GND -> GND
- LED22 pad 1: +5V -> +5V_LED
- LED22 pad 4: /LED_GND -> GND
- LED23 pad 1: +5V -> +5V_LED
- LED23 pad 4: /LED_GND -> GND
- LED24 pad 1: +5V -> +5V_LED
- LED24 pad 4: /LED_GND -> GND
- LED25 pad 1: +5V -> +5V_LED
- LED25 pad 4: /LED_GND -> GND
- LED26 pad 1: +5V -> +5V_LED
- LED26 pad 4: /LED_GND -> GND
- LED27 pad 1: +5V -> +5V_LED
- LED27 pad 4: /LED_GND -> GND
- LED28 pad 1: +5V -> +5V_LED
- LED28 pad 4: /LED_GND -> GND
- LED29 pad 1: +5V -> +5V_LED
- LED29 pad 4: /LED_GND -> GND
- LED3 pad 1: +5V -> +5V_LED
- LED3 pad 4: /LED_GND -> GND
- LED30 pad 1: +5V -> +5V_LED
- LED30 pad 4: /LED_GND -> GND
- LED31 pad 1: +5V -> +5V_LED
- LED31 pad 4: /LED_GND -> GND
- LED32 pad 1: +5V -> +5V_LED
- LED32 pad 4: /LED_GND -> GND
- LED33 pad 1: +5V -> +5V_LED
- LED33 pad 4: /LED_GND -> GND
- LED34 pad 1: +5V -> +5V_LED
- LED34 pad 4: /LED_GND -> GND
- LED35 pad 1: +5V -> +5V_LED
- LED35 pad 4: /LED_GND -> GND
- LED36 pad 1: +5V -> +5V_LED
- LED36 pad 4: /LED_GND -> GND
- LED37 pad 1: +5V -> +5V_LED
- LED37 pad 4: /LED_GND -> GND
- LED38 pad 1: +5V -> +5V_LED
- LED38 pad 4: /LED_GND -> GND
- LED39 pad 1: +5V -> +5V_LED
- LED39 pad 4: /LED_GND -> GND
- LED4 pad 1: +5V -> +5V_LED
- LED4 pad 4: /LED_GND -> GND
- LED40 pad 1: +5V -> +5V_LED
- LED40 pad 4: /LED_GND -> GND
- LED41 pad 1: +5V -> +5V_LED
- LED41 pad 4: /LED_GND -> GND
- LED42 pad 1: +5V -> +5V_LED
- LED42 pad 4: /LED_GND -> GND
- LED43 pad 1: +5V -> +5V_LED
- LED43 pad 4: /LED_GND -> GND
- LED44 pad 1: +5V -> +5V_LED
- LED44 pad 4: /LED_GND -> GND
- LED45 pad 1: +5V -> +5V_LED
- LED45 pad 4: /LED_GND -> GND
- LED46 pad 1: +5V -> +5V_LED
- LED46 pad 4: /LED_GND -> GND
- LED47 pad 1: +5V -> +5V_LED
- LED47 pad 4: /LED_GND -> GND
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Routing:
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Other:
- board size 347.9 x 125.8 mm -> 3.6 x 3.3 mm

Commit message: progress idk. western duplex matrix. stuff.
Parts:
- removed the D88 at (46.4, 49.8)
- removed the D88 at (76.5, 49.5)
- removed the Q1 at (50.5, 52.2)
- removed the Q1 at (66.7, 52.4)
- removed Q3: Q_PMOS, Package_TO_SOT_SMD:SOT-23_Handsoldering
- removed R1: 806k, Resistor_SMD:R_0402_1005Metric_Pad0.72x0.64mm_HandSolder
- removed R2: 2M, Resistor_SMD:R_0402_1005Metric_Pad0.72x0.64mm_HandSolder
- removed R3, R4, R5: 4.7kΩ, Capacitor_SMD:C_0402_1005Metric_Pad0.74x0.62mm_HandSolder
- removed the REF** at (292.9, 104.8)
- removed the REF** at (50.0, 123.8)
- removed TP3, TP4: TestPoint, TestPoint:TestPoint_Pad_D1.5mm
- removed U4: PCA9555PW, Package_SO:TSSOP-24_4.4x7.8mm_P0.65mm
- added D88: D, Diode_SMD:D_SOD-323_HandSoldering, F.Cu at (-25.4, 27.6)
- added D90: D, Diode_SMD:D_SOD-323_HandSoldering, F.Cu at (-110.4, 83.2)
- added D91: D, Diode_SMD:D_SOD-323_HandSoldering, F.Cu at (-110.4, 86.1)
- added D92: D, Diode_SMD:D_SOD-323_HandSoldering, F.Cu at (351.0, 102.3)
- added J2: Conn_01x04_MountingPin, Connector_JST:JST_SH_BM04B-SRSS-TB_1x04-1MP_P1.00mm_Vertical, F.Cu at (-83.9, 58.3)
- added Q1: AO3401A, Package_TO_SOT_SMD:SOT-23, F.Cu at (-59.0, 51.3)
- added Q2: AO3401A, Package_TO_SOT_SMD:SOT-23, F.Cu at (-59.0, 55.7)
- added REF**: STAB_MX_2.25u, marbastlib-mx:STAB_MX_2.25u, F.Cu at (292.9, 104.8)
- C2, D89, L1, TP1, TP2, U3: moved to F.Cu
- SW34, SW47: footprint marbastlib-mx:SW_MX_HS_CPG151101S11_1u -> marbastlib-mx:SW_MX_HS_CPG151101S11_1.5u
- SW35, SW48: footprint marbastlib-mx:SW_MX_HS_CPG151101S11_1.5u -> marbastlib-mx:SW_MX_HS_CPG151101S11_1u
- SW51: footprint marbastlib-mx:SW_MX_HS_CPG151101S11_1u -> marbastlib-mx:SW_MX_HS_CPG151101S11_1.75u
- SW52: footprint marbastlib-mx:SW_MX_HS_CPG151101S11_1.75u -> marbastlib-mx:SW_MX_HS_CPG151101S11_1u
- SW77, SW81: footprint marbastlib-mx:SW_MX_HS_CPG151101S11_1u -> marbastlib-mx:SW_MX_HS_CPG151101S11_1.25u
- SW80, SW85: footprint marbastlib-mx:SW_MX_HS_CPG151101S11_1.25u -> marbastlib-mx:SW_MX_HS_CPG151101S11_1u
- U1: value XIAO-nRF52840-SMD -> Guilty Devboard Xrd; footprint OPL:XIAO-nRF52840-SMD -> xrd-lib:Guilty Devboard Xrd - SMD; moved to F.Cu
- moved G*** 200.0 mm to (184.1, 339.8)
- moved G*** 200.0 mm to (316.5, 332.2)
- moved TP1 116.3 mm to (-30.0, 28.1)
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Connections:
- D1 pad 1: /ROW4 -> /ROW0
- D10 pad 1: /ROW8 -> /ROW0
- D11 pad 1: /ROW8 -> /ROW1
- D12 pad 1: /ROW7 -> /ROW0
- D13 pad 1: /ROW6 -> /ROW1
- D14 pad 1: /ROW5 -> /ROW0
- D15 pad 1: /ROW4 -> /ROW1
- D16 pad 1: /ROW3 -> /ROW0
- D18 pad 1: /ROW0 -> /ROW3
- D19 pad 1: /ROW1 -> /ROW2
- D20 pad 1: /ROW0 -> /ROW3
- D21 pad 1: /ROW1 -> /ROW2
- D22 pad 1: /ROW2 -> /ROW3
- D23 pad 1: /ROW3 -> /ROW2
- D24 pad 1: /ROW4 -> /ROW3
- D25 pad 1: /ROW5 -> /ROW2
- D26 pad 1: /ROW6 -> /ROW3
- D27 pad 1: /ROW7 -> /ROW2
- D28 pad 1: /ROW8 -> /ROW3
- D30 pad 1: /ROW4 -> /ROW3
- D31 pad 1: /ROW3 -> /ROW2
- D32 pad 1: /ROW7 -> /ROW3
- D33 pad 1: /ROW6 -> /ROW2
- D34 pad 1: /ROW5 -> /ROW4
- D35 pad 1: /ROW0 -> unconnected-(D35-K-Pad1)
- D36 pad 1: /ROW1 -> /ROW4
- D37 pad 1: /ROW8 -> unconnected-(D37-K-Pad1)
- D38 pad 1: /ROW0 -> /ROW4
- D39 pad 1: /ROW1 -> unconnected-(D39-K-Pad1)
- D4 pad 1: /ROW2 -> /ROW0
- D40 pad 1: /ROW7 -> /ROW4
- D41 pad 1: /ROW8 -> unconnected-(D41-K-Pad1)
- D42 pad 1: /ROW5 -> /ROW4
- D43 pad 1: /ROW6 -> unconnected-(D43-K-Pad1)
- D45 pad 1: /ROW2 -> unconnected-(D45-K-Pad1)
- D46 pad 1: /ROW3 -> /ROW4
- D47 pad 1: /ROW3 -> unconnected-(D47-K-Pad1)
- D48 pad 1: /ROW2 -> /ROW4
- D49 pad 1: /ROW7 -> /ROW5
- D5 pad 1: /ROW3 -> /ROW1
- D50 pad 1: /ROW6 -> /ROW4
- D51 pad 1: /ROW5 -> /ROW6
- D52 pad 1: /ROW0 -> /ROW7
- D53 pad 1: /ROW1 -> /ROW6
- D54 pad 1: /ROW4 -> /ROW7
- D55 pad 1: /ROW8 -> /ROW6
- D56 pad 1: /ROW0 -> /ROW7
- D57 pad 1: /ROW1 -> /ROW6
- D58 pad 1: /ROW5 -> /ROW7
- D6 pad 1: /ROW4 -> /ROW0
- D61 pad 1: /ROW8 -> /ROW6
- D62 pad 1: /ROW2 -> /ROW7
- D63 pad 1: /ROW3 -> /ROW6
- D64 pad 1: /ROW4 -> /ROW8
- D65 pad 1: /ROW0 -> /ROW9
- D66 pad 1: /ROW1 -> /ROW8
- D67 pad 1: /ROW4 -> /ROW9
- D68 pad 1: /ROW5 -> /ROW8
- D69 pad 1: /ROW6 -> /ROW9
- D7 pad 1: /ROW5 -> /ROW1
- D70 pad 1: /ROW7 -> /ROW8
- D71 pad 1: /ROW8 -> /ROW9
- D72 pad 1: /ROW3 -> /ROW8
- D73 pad 1: /ROW2 -> /ROW9
- D74 pad 1: /ROW2 -> /ROW8
- D75 pad 1: /ROW3 -> /ROW9
- D76 pad 1: /ROW8 -> /ROW9
- D77 pad 1: /ROW4 -> /ROW10
- D78 pad 1: /ROW0 -> /ROW11
- D79 pad 1: /ROW1 -> /ROW10
- D8 pad 1: /ROW6 -> /ROW0
- D80 pad 1: /ROW5 -> /ROW11
- D81 pad 1: /ROW6 -> /ROW10
- D82 pad 1: /ROW7 -> /ROW11
- D83 pad 1: /ROW7 -> /ROW10
- D84 pad 1: /ROW2 -> /ROW11
- D85 pad 1: /ROW3 -> /ROW10
- D86 pad 1: /ROW6 -> /ROW11
- D87 pad 1: /ROW5 -> /ROW10
- D9 pad 1: /ROW7 -> /ROW1
- LED17 pad 3: Net-(LED16-DOUT) -> Net-(LED17-DIN)
- LED18 pad 1: +5V_LED -> Net-(LED18-VDD)
- LED18 pad 2: Net-(LED18-DOUT) -> Net-(LED17-DIN)
- LED18 pad 3: Net-(LED17-DOUT) -> Net-(LED18-DIN)
- LED19 pad 1: +5V_LED -> Net-(LED19-VDD)
- LED19 pad 2: Net-(LED19-DOUT) -> Net-(LED18-DIN)
- LED19 pad 3: Net-(LED18-DOUT) -> Net-(LED19-DIN)
- LED20 pad 1: +5V_LED -> Net-(LED20-VDD)
- LED20 pad 2: Net-(LED20-DOUT) -> Net-(LED19-DIN)
- LED20 pad 3: Net-(LED19-DOUT) -> Net-(LED20-DIN)
- LED21 pad 1: +5V_LED -> Net-(LED21-VDD)
- LED21 pad 2: Net-(LED21-DOUT) -> Net-(LED20-DIN)
- LED21 pad 3: Net-(LED20-DOUT) -> Net-(LED21-DIN)
- LED22 pad 1: +5V_LED -> Net-(LED22-VDD)
- LED22 pad 2: Net-(LED22-DOUT) -> Net-(LED21-DIN)
- LED22 pad 3: Net-(LED21-DOUT) -> Net-(LED22-DIN)
- LED23 pad 1: +5V_LED -> Net-(LED23-VDD)
- LED23 pad 2: Net-(LED23-DOUT) -> Net-(LED22-DIN)
- LED23 pad 3: Net-(LED22-DOUT) -> Net-(LED23-DIN)
- LED24 pad 1: +5V_LED -> Net-(LED24-VDD)
- LED24 pad 2: Net-(LED24-DOUT) -> Net-(LED23-DIN)
- LED24 pad 3: Net-(LED23-DOUT) -> Net-(LED24-DIN)
- LED25 pad 1: +5V_LED -> Net-(LED25-VDD)
- LED25 pad 2: Net-(LED25-DOUT) -> Net-(LED24-DIN)
- LED25 pad 3: Net-(LED24-DOUT) -> Net-(LED25-DIN)
- LED26 pad 1: +5V_LED -> Net-(LED26-VDD)
- LED26 pad 2: Net-(LED26-DOUT) -> Net-(LED25-DIN)
- LED26 pad 3: Net-(LED25-DOUT) -> Net-(LED26-DIN)
- LED27 pad 1: +5V_LED -> Net-(LED27-VDD)
- LED27 pad 2: Net-(LED27-DOUT) -> Net-(LED26-DIN)
- LED27 pad 3: Net-(LED26-DOUT) -> Net-(LED27-DIN)
- LED28 pad 1: +5V_LED -> Net-(LED28-VDD)
- LED28 pad 2: Net-(LED28-DOUT) -> Net-(LED27-DIN)
- LED28 pad 3: Net-(LED27-DOUT) -> Net-(LED28-DIN)
- LED29 pad 1: +5V_LED -> Net-(LED29-VDD)
- LED29 pad 2: Net-(LED29-DOUT) -> Net-(LED28-DIN)
- LED29 pad 3: Net-(LED28-DOUT) -> Net-(LED29-DIN)
- LED30 pad 1: +5V_LED -> Net-(LED30-VDD)
- LED30 pad 2: Net-(LED30-DOUT) -> Net-(LED29-DIN)
- LED30 pad 3: Net-(LED29-DOUT) -> Net-(LED30-DIN)
- LED31 pad 1: +5V_LED -> Net-(LED31-VDD)
- LED31 pad 2: Net-(LED31-DOUT) -> Net-(LED30-DIN)
- LED31 pad 3: Net-(LED30-DOUT) -> Net-(LED31-DIN)
- LED32 pad 1: +5V_LED -> Net-(LED32-VDD)
- LED32 pad 2: Net-(LED32-DOUT) -> Net-(LED31-DIN)
- LED32 pad 3: Net-(LED31-DOUT) -> Net-(LED32-DIN)
- LED33 pad 2: Net-(LED33-DOUT) -> Net-(LED32-DIN)
- LED33 pad 3: Net-(LED32-DOUT) -> Net-(LED16-DOUT)
- LED34 pad 3: Net-(LED33-DOUT) -> Net-(LED17-DOUT)
- LED35 pad 1: +5V_LED -> Net-(LED18-VDD)
- LED35 pad 4: GND -> Net-(LED35-VSS)
- LED36 pad 1: +5V_LED -> Net-(LED19-VDD)
- LED36 pad 4: GND -> Net-(LED36-VSS)
- LED37 pad 1: +5V_LED -> Net-(LED20-VDD)
- LED37 pad 4: GND -> Net-(LED37-VSS)
- LED38 pad 1: +5V_LED -> Net-(LED21-VDD)
- LED38 pad 4: GND -> Net-(LED38-VSS)
- LED39 pad 1: +5V_LED -> Net-(LED22-VDD)
- LED39 pad 4: GND -> Net-(LED39-VSS)
- LED40 pad 1: +5V_LED -> Net-(LED23-VDD)
- LED40 pad 4: GND -> Net-(LED40-VSS)
- LED41 pad 1: +5V_LED -> Net-(LED24-VDD)
- LED41 pad 4: GND -> Net-(LED41-VSS)
- LED42 pad 1: +5V_LED -> Net-(LED25-VDD)
- LED42 pad 4: GND -> Net-(LED42-VSS)
- LED43 pad 1: +5V_LED -> Net-(LED26-VDD)
- LED43 pad 4: GND -> Net-(LED43-VSS)
- LED44 pad 1: +5V_LED -> Net-(LED27-VDD)
- LED44 pad 4: GND -> Net-(LED44-VSS)
- LED45 pad 1: +5V_LED -> Net-(LED28-VDD)
- LED45 pad 4: GND -> Net-(LED45-VSS)
- LED46 pad 1: +5V_LED -> Net-(LED29-VDD)
- LED47 pad 1: +5V_LED -> Net-(LED30-VDD)
- LED47 pad 4: GND -> unconnected-(LED47-VSS-Pad4)
- LED48 pad 1: +5V_LED -> Net-(LED31-VDD)
- LED48 pad 4: GND -> unconnected-(LED48-VSS-Pad4)
- LED49 pad 1: +5V_LED -> Net-(LED32-VDD)
- LED49 pad 4: GND -> unconnected-(LED49-VSS-Pad4)
- LED50 pad 4: GND -> unconnected-(LED50-VSS-Pad4)
- LED51 pad 3: Net-(LED50-DOUT) -> Net-(LED51-DIN)
- LED52 pad 1: +5V_LED -> Net-(LED52-VDD)
- LED52 pad 2: Net-(LED52-DOUT) -> Net-(LED51-DIN)
- LED52 pad 3: Net-(LED51-DOUT) -> Net-(LED52-DIN)
- LED52 pad 4: GND -> Net-(LED35-VSS)
- LED53 pad 1: +5V_LED -> Net-(LED53-VDD)
- LED53 pad 2: Net-(LED53-DOUT) -> Net-(LED52-DIN)
- LED53 pad 3: Net-(LED52-DOUT) -> Net-(LED53-DIN)
- LED53 pad 4: GND -> Net-(LED36-VSS)
- LED54 pad 1: +5V_LED -> Net-(LED54-VDD)
- LED54 pad 2: Net-(LED54-DOUT) -> Net-(LED53-DIN)
- LED54 pad 3: Net-(LED53-DOUT) -> Net-(LED54-DIN)
- LED54 pad 4: GND -> Net-(LED37-VSS)
- LED55 pad 1: +5V_LED -> Net-(LED55-VDD)
- LED55 pad 2: Net-(LED55-DOUT) -> Net-(LED54-DIN)
- LED55 pad 3: Net-(LED54-DOUT) -> Net-(LED55-DIN)
- LED55 pad 4: GND -> Net-(LED38-VSS)
- LED56 pad 1: +5V_LED -> Net-(LED56-VDD)
- LED56 pad 2: Net-(LED56-DOUT) -> Net-(LED55-DIN)
- LED56 pad 3: Net-(LED55-DOUT) -> Net-(LED56-DIN)
- LED56 pad 4: GND -> Net-(LED39-VSS)
- LED57 pad 1: +5V_LED -> Net-(LED57-VDD)
- LED57 pad 2: Net-(LED57-DOUT) -> Net-(LED56-DIN)
- LED57 pad 3: Net-(LED56-DOUT) -> Net-(LED57-DIN)
- LED57 pad 4: GND -> Net-(LED40-VSS)
- LED58 pad 1: +5V_LED -> Net-(LED58-VDD)
- LED58 pad 2: Net-(LED58-DOUT) -> Net-(LED57-DIN)
- LED58 pad 3: Net-(LED57-DOUT) -> Net-(LED58-DIN)
- LED58 pad 4: GND -> Net-(LED41-VSS)
- LED59 pad 1: +5V_LED -> Net-(LED59-VDD)
- LED59 pad 2: Net-(LED59-DOUT) -> Net-(LED58-DIN)
- LED59 pad 3: Net-(LED58-DOUT) -> Net-(LED59-DIN)
- LED59 pad 4: GND -> Net-(LED42-VSS)
- LED60 pad 1: +5V_LED -> Net-(LED60-VDD)
- LED60 pad 2: Net-(LED60-DOUT) -> Net-(LED59-DIN)
- LED60 pad 3: Net-(LED59-DOUT) -> Net-(LED60-DIN)
- LED60 pad 4: GND -> Net-(LED43-VSS)
- LED61 pad 1: +5V_LED -> Net-(LED61-VDD)
- LED61 pad 2: Net-(LED61-DOUT) -> Net-(LED60-DIN)
- LED61 pad 3: Net-(LED60-DOUT) -> Net-(LED61-DIN)
- LED61 pad 4: GND -> Net-(LED44-VSS)
- LED62 pad 1: +5V_LED -> Net-(LED62-VDD)
- LED62 pad 2: Net-(LED62-DOUT) -> Net-(LED61-DIN)
- LED62 pad 3: Net-(LED61-DOUT) -> Net-(LED62-DIN)
- LED62 pad 4: GND -> Net-(LED45-VSS)
- LED63 pad 2: Net-(LED63-DOUT) -> Net-(LED62-DIN)
- LED63 pad 3: Net-(LED62-DOUT) -> Net-(LED50-DOUT)
- LED64 pad 3: Net-(LED63-DOUT) -> Net-(LED51-DOUT)
- LED65 pad 1: +5V_LED -> Net-(LED52-VDD)
- LED66 pad 1: +5V_LED -> Net-(LED53-VDD)
- LED67 pad 1: +5V_LED -> Net-(LED54-VDD)
- LED68 pad 1: +5V_LED -> Net-(LED55-VDD)
- LED69 pad 1: +5V_LED -> Net-(LED56-VDD)
- LED70 pad 1: +5V_LED -> Net-(LED57-VDD)
- LED71 pad 1: +5V_LED -> Net-(LED58-VDD)
- LED72 pad 1: +5V_LED -> Net-(LED59-VDD)
- LED73 pad 1: +5V_LED -> Net-(LED60-VDD)
- LED74 pad 1: +5V_LED -> Net-(LED61-VDD)
- LED75 pad 1: +5V_LED -> Net-(LED62-VDD)
- LED77 pad 2: Net-(LED77-DOUT) -> unconnected-(LED77-DOUT-Pad2)
- LED77 pad 3: Net-(LED76-DOUT) -> Net-(LED77-DIN)
- LED78 pad 2: Net-(LED78-DOUT) -> Net-(LED77-DIN)
- LED78 pad 3: Net-(LED77-DOUT) -> Net-(LED78-DIN)
- LED79 pad 2: Net-(LED79-DOUT) -> Net-(LED78-DIN)
- LED79 pad 3: Net-(LED78-DOUT) -> Net-(LED79-DIN)
- LED80 pad 2: Net-(LED80-DOUT) -> Net-(LED79-DIN)
- LED80 pad 3: Net-(LED79-DOUT) -> Net-(LED80-DIN)
- LED81 pad 2: Net-(LED81-DOUT) -> Net-(LED80-DIN)
- LED81 pad 3: Net-(LED80-DOUT) -> Net-(LED81-DIN)
- LED82 pad 2: Net-(LED82-DOUT) -> Net-(LED81-DIN)
- LED82 pad 3: Net-(LED81-DOUT) -> Net-(LED82-DIN)
- LED83 pad 2: Net-(LED83-DOUT) -> Net-(LED82-DIN)
- LED83 pad 3: Net-(LED82-DOUT) -> Net-(LED83-DIN)
- LED84 pad 2: Net-(LED84-DOUT) -> Net-(LED83-DIN)
- LED84 pad 3: Net-(LED83-DOUT) -> Net-(LED84-DIN)
- LED85 pad 2: Net-(LED85-DOUT) -> Net-(LED84-DIN)
- LED85 pad 3: Net-(LED84-DOUT) -> Net-(LED85-DIN)
- LED86 pad 2: Net-(LED86-DOUT) -> Net-(LED85-DIN)
- LED86 pad 3: Net-(LED85-DOUT) -> Net-(LED86-DIN)
- LED87 pad 2: unconnected-(LED87-DOUT-Pad2) -> Net-(LED86-DIN)
- LED87 pad 3: Net-(LED86-DOUT) -> Net-(LED76-DOUT)
- SW10 pad 1: /COL9 -> /COL5
- SW11 pad 1: /COL8 -> /COL5
- SW12 pad 1: /COL8 -> /COL6
- SW13 pad 1: /COL8 -> /COL6
- SW14 pad 1: /COL8 -> /COL7
- SW15 pad 1: /COL8 -> /COL7
- SW17 pad 1: /COL8 -> /COL0
- SW18 pad 1: /COL8 -> /COL0
- SW19 pad 1: /COL8 -> /COL1
- SW2 pad 1: /COL9 -> /COL1
- SW20 pad 1: /COL7 -> /COL1
- SW21 pad 1: /COL7 -> /COL2
- SW22 pad 1: /COL7 -> /COL2
- SW23 pad 1: /COL7 -> /COL3
- SW24 pad 1: /COL7 -> /COL3
- SW25 pad 1: /COL7 -> /COL4
- SW26 pad 1: /COL7 -> /COL4
- SW27 pad 1: /COL7 -> /COL5
- SW28 pad 1: /COL7 -> /COL5
- SW3 pad 1: /COL9 -> /COL1
- SW31 pad 1: /COL6 -> /COL7
- SW32 pad 1: /COL6 -> /COL7
- SW33 pad 1: /COL6 -> /COL8
- SW34 pad 1: /COL6 -> /COL0
- SW35 pad 1: /COL6 -> /COL0
- SW36 pad 1: /COL6 -> /COL1
- SW37 pad 1: /COL6 -> /COL1
- SW38 pad 1: /COL5 -> /COL2
- SW39 pad 1: /COL5 -> /COL2
- SW4 pad 1: /COL9 -> /COL2
- SW40 pad 1: /COL5 -> /COL3
- SW41 pad 1: /COL5 -> /COL3
- SW42 pad 1: /COL5 -> /COL4
- SW43 pad 1: /COL5 -> /COL4
- SW46 pad 1: /COL5 -> /COL6
- SW47 pad 1: /COL4 -> /COL6
- SW48 pad 1: /COL4 -> /COL7
- SW49 pad 1: /COL4 -> /COL7
- SW5 pad 1: /COL9 -> /COL2
- SW50 pad 1: /COL4 -> /COL8
- SW51 pad 1: /COL4 -> /COL0
- SW52 pad 1: /COL4 -> /COL0
- SW53 pad 1: /COL4 -> /COL1
- SW54 pad 1: /COL4 -> /COL1
- SW55 pad 1: /COL4 -> /COL2
- SW56 pad 1: /COL3 -> /COL2
- SW59 pad 1: /COL3 -> /COL4
- SW6 pad 1: /COL9 -> /COL3
- SW60 pad 1: /COL3 -> /COL4
- SW61 pad 1: /COL3 -> /COL5
- SW62 pad 1: /COL3 -> /COL5
- SW63 pad 1: /COL3 -> /COL6
- SW64 pad 1: /COL3 -> /COL0
- SW65 pad 1: /COL2 -> /COL0
- SW66 pad 1: /COL2 -> /COL1
- SW67 pad 1: /COL2 -> /COL1
- SW7 pad 1: /COL9 -> /COL3
- SW70 pad 1: /COL2 -> /COL3
- SW71 pad 1: /COL2 -> /COL3
- SW72 pad 1: /COL2 -> /COL4
- SW73 pad 1: /COL2 -> /COL4
- SW74 pad 1: /COL1 -> /COL5
- SW75 pad 1: /COL1 -> /COL5
- SW76 pad 1: /COL1 -> /COL7
- SW77 pad 1: /COL1 -> /COL0
- SW78 pad 1: /COL1 -> /COL0
- SW8 pad 1: /COL9 -> /COL4
- SW80 pad 1: /COL1 -> /COL2
- SW81 pad 1: /COL1 -> /COL4
- SW82 pad 1: /COL1 -> /COL4
- SW83 pad 1: /COL0 -> /COL5
- SW84 pad 1: /COL0 -> /COL5
- SW85 pad 1: /COL0 -> /COL7
- SW86 pad 1: /COL0 -> /COL7
- SW87 pad 1: /COL0 -> /COL8
- SW89 pad S1: /EC11_SW -> /COL8
- SW89 pad S2: GND -> /EC11_SW2
- SW9 pad 1: /COL9 -> /COL4
- U1 pad 1: /BT_PIN -> /COL4
- U1 pad 10: /COL8 -> +3V3
- U1 pad 11: /COL7 -> /COL8
- U1 pad 12: +3V3 -> /COL7
- U1 pad 13: GND -> /EC11_A
- U1 pad 14: +5V_USB -> /EC11_B
- U1 pad 15: /VBAT -> /COL3
- U1 pad 16: GND -> /COL1
- U1 pad 17: Net-(U1-NFC1) -> /ROW11
- U1 pad 18: Net-(U1-NFC2) -> /ROW9
- U1 pad 19: unconnected-(U1-PA31_SWDIO-Pad19) -> /ROW7
- U1 pad 2: /EC11_SW -> /COL2
- U1 pad 20: unconnected-(U1-PA30_SWCLK-Pad20) -> /ROW5
- U1 pad 21: unconnected-(U1-RESET-Pad21) -> /COL6
- U1 pad 22: unconnected-(U1-GND-Pad22) -> /COL5
- U1 pad 3: /EC11_B -> /COL0
- U1 pad 4: /EC11_A -> /ROW10
- U1 pad 5: /I2C_SDA -> /ROW8
- U1 pad 6: /I2C_SCL -> /ROW6
- U1 pad 7: /LED_ENABLE -> /ROW4
- U1 pad 8: Net-(U1-P1.12_D7_RX) -> +5V_USB
- U1 pad 9: /COL9 -> GND
- U2 pad 1: Net-(U1-P1.12_D7_RX) -> Net-(U1-D17_SCK1)
- U2 pad 2: Net-(U1-P1.12_D7_RX) -> Net-(U1-D17_SCK1)
- U5 pad 1: /LED_ENABLE -> Net-(D90-K)
- U5 pad 2: /LED_ENABLE -> Net-(D90-K)
Routing:
- net GND: track 1322.0 -> 0.00 mm, vias 3 -> 0
- net +5V_LED: track 1087.9 -> 0.00 mm, vias 2 -> 0
- net /COL1: track 574.9 -> 0.00 mm
- net /COL3: track 533.4 -> 0.00 mm
- net /COL5: track 457.2 -> 0.00 mm
- net /COL4: track 350.0 -> 0.00 mm
- net Net-(LED50-DOUT): track 348.8 -> 0.00 mm, vias 2 -> 0
- net /COL0: track 321.5 -> 0.00 mm
- net /COL2: track 304.8 -> 0.00 mm
- net /COL7: track 200.2 -> 34.5 mm, vias 1 -> 0
- net /COL6: track 158.9 -> 0.00 mm
- net /COL9: track 147.9 -> 0.00 mm
- net /COL8: track 171.7 -> 58.2 mm, vias 2 -> 0
- net +3V3: track 107.9 -> 0.00 mm, vias 1 -> 0
- net /I2C_SDA: track 91.1 -> 0.00 mm, vias 1 -> 0
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Other:
- board size 3.6 x 3.3 mm -> 347.8 x 124 mm

Commit message: finish schematic and routing
Parts:
- removed C2: 10μF, Capacitor_SMD:C_0603_1608Metric_Pad1.08x0.95mm_HandSolder
- removed D90, D91: D, Diode_SMD:D_SOD-323_HandSoldering
- removed L1: 15μH, Inductor_SMD_Wurth:L_Wurth_WE-LQSH-4020
- removed Q1, Q2: AO3401A, Package_TO_SOT_SMD:SOT-23
- removed U5: 74LV1T08GW, Package_TO_SOT_SMD:SOT-353_SC-70-5
- added C1: 0.1uF, Capacitor_SMD:C_0603_1608Metric, F.Cu at (56.3, 51.9)
- added C10: 4.7uF, Capacitor_SMD:C_0603_1608Metric, F.Cu at (57.7, 51.9)
- added C20: 22uF, Capacitor_SMD:C_0603_1608Metric, F.Cu at (65.5, 51.5)
- added C21: 22uF, Capacitor_SMD:C_0603_1608Metric, F.Cu at (36.2, 56.3)
- added C22: 1uF, Capacitor_SMD:C_0603_1608Metric, F.Cu at (59.2, 51.9)
- added C23: 22uF, Capacitor_SMD:C_0603_1608Metric, F.Cu at (54.1, 50.7)
- added L2: 2.2uH, Inductor_SMD:L_0805_2012Metric, F.Cu at (60.8, 51.6)
- added R1: 1M, Resistor_SMD:R_0603_1608Metric, F.Cu at (53.3, 52.9)
- added U8: MIC2876-5.0YMT-TR, easyeda2kicad:UDFN-8_L2.0-W2.0-P0.50-BL-EP, F.Cu at (63.3, 51.5)
- TP1, TP2: moved to B.Cu
- U3: value TPS613222ADBV -> SiP32408; footprint Package_TO_SOT_SMD:SOT-23-5 -> gpxxacpy:UDFN-4-1EP_1.2x1.6mm_P0.5mm_EP0.86x0.5mm
- moved G*** 200.0 mm to (184.1, 139.8)
- moved G*** 200.0 mm to (316.5, 132.2)
- moved J2 116.2 mm to (32.1, 52.4), turned to 90 degrees
- moved U2 98.5 mm to (67.6, 49.2), turned to -90 degrees
- moved U3 91.8 mm to (54.8, 52.4), turned to -90 degrees
- moved TP2 90.3 mm to (59.0, 47.5), turned to -90 degrees
- moved D89 90.2 mm to (61.6, 54.3)
- moved TP1 87.6 mm to (55.5, 47.5), turned to -90 degrees
- moved D88 87.2 mm to (57.6, 54.3), turned to 180 degrees
- moved D92 22.3 mm to (372.5, 96.5), turned to 0 degrees
- turned LED1 to 0 degrees
- turned LED10 to 0 degrees
- turned LED11 to 0 degrees
- turned LED12 to 0 degrees
- turned LED13 to 0 degrees
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Connections:
- D35 pad 1: unconnected-(D35-K-Pad1) -> /ROW5
- D37 pad 1: unconnected-(D37-K-Pad1) -> /ROW5
- D39 pad 1: unconnected-(D39-K-Pad1) -> /ROW5
- D41 pad 1: unconnected-(D41-K-Pad1) -> /ROW5
- D43 pad 1: unconnected-(D43-K-Pad1) -> /ROW5
- D45 pad 1: unconnected-(D45-K-Pad1) -> /ROW5
- D47 pad 1: unconnected-(D47-K-Pad1) -> /ROW5
- J2 pad 4: Net-(J2-MountPin) -> GND
- J2 pad MP: Net-(J2-MountPin) -> GND
- LED1 pad 1: +5V_LED -> +5V
- LED10 pad 1: +5V_LED -> +5V
- LED11 pad 1: +5V_LED -> +5V
- LED12 pad 1: +5V_LED -> +5V
- LED13 pad 1: +5V_LED -> +5V
- LED14 pad 1: +5V_LED -> +5V
- LED15 pad 1: +5V_LED -> +5V
- LED16 pad 1: +5V_LED -> +5V
- LED17 pad 1: +5V_LED -> +5V
- LED18 pad 1: Net-(LED18-VDD) -> +5V
- LED19 pad 1: Net-(LED19-VDD) -> +5V
- LED2 pad 1: +5V_LED -> +5V
- LED20 pad 1: Net-(LED20-VDD) -> +5V
- LED21 pad 1: Net-(LED21-VDD) -> +5V
- LED22 pad 1: Net-(LED22-VDD) -> +5V
- LED23 pad 1: Net-(LED23-VDD) -> +5V
- LED24 pad 1: Net-(LED24-VDD) -> +5V
- LED25 pad 1: Net-(LED25-VDD) -> +5V
- LED26 pad 1: Net-(LED26-VDD) -> +5V
- LED27 pad 1: Net-(LED27-VDD) -> +5V
- LED28 pad 1: Net-(LED28-VDD) -> +5V
- LED29 pad 1: Net-(LED29-VDD) -> +5V
- LED3 pad 1: +5V_LED -> +5V
- LED30 pad 1: Net-(LED30-VDD) -> +5V
- LED31 pad 1: Net-(LED31-VDD) -> +5V
- LED32 pad 1: Net-(LED32-VDD) -> +5V
- LED33 pad 1: +5V_LED -> +5V
- LED34 pad 1: +5V_LED -> +5V
- LED35 pad 1: Net-(LED18-VDD) -> +5V
- LED35 pad 4: Net-(LED35-VSS) -> GND
- LED36 pad 1: Net-(LED19-VDD) -> +5V
- LED36 pad 4: Net-(LED36-VSS) -> GND
- LED37 pad 1: Net-(LED20-VDD) -> +5V
- LED37 pad 4: Net-(LED37-VSS) -> GND
- LED38 pad 1: Net-(LED21-VDD) -> +5V
- LED38 pad 4: Net-(LED38-VSS) -> GND
- LED39 pad 1: Net-(LED22-VDD) -> +5V
- LED39 pad 4: Net-(LED39-VSS) -> GND
- LED4 pad 1: +5V_LED -> +5V
- LED40 pad 1: Net-(LED23-VDD) -> +5V
- LED40 pad 4: Net-(LED40-VSS) -> GND
- LED41 pad 1: Net-(LED24-VDD) -> +5V
- LED41 pad 4: Net-(LED41-VSS) -> GND
- LED42 pad 1: Net-(LED25-VDD) -> +5V
- LED42 pad 4: Net-(LED42-VSS) -> GND
- LED43 pad 1: Net-(LED26-VDD) -> +5V
- LED43 pad 4: Net-(LED43-VSS) -> GND
- LED44 pad 1: Net-(LED27-VDD) -> +5V
- LED44 pad 4: Net-(LED44-VSS) -> GND
- LED45 pad 1: Net-(LED28-VDD) -> +5V
- LED45 pad 4: Net-(LED45-VSS) -> GND
- LED46 pad 1: Net-(LED29-VDD) -> +5V
- LED47 pad 1: Net-(LED30-VDD) -> +5V
- LED47 pad 4: unconnected-(LED47-VSS-Pad4) -> GND
- LED48 pad 1: Net-(LED31-VDD) -> +5V
- LED48 pad 4: unconnected-(LED48-VSS-Pad4) -> GND
- LED49 pad 1: Net-(LED32-VDD) -> +5V
- LED49 pad 4: unconnected-(LED49-VSS-Pad4) -> GND
- LED5 pad 1: +5V_LED -> +5V
- LED50 pad 1: +5V_LED -> +5V
- LED50 pad 4: unconnected-(LED50-VSS-Pad4) -> GND
- LED51 pad 1: +5V_LED -> +5V
- LED52 pad 1: Net-(LED52-VDD) -> +5V
- LED52 pad 4: Net-(LED35-VSS) -> GND
- LED53 pad 1: Net-(LED53-VDD) -> +5V
- LED53 pad 4: Net-(LED36-VSS) -> GND
- LED54 pad 1: Net-(LED54-VDD) -> +5V
- LED54 pad 4: Net-(LED37-VSS) -> GND
- LED55 pad 1: Net-(LED55-VDD) -> +5V
- LED55 pad 4: Net-(LED38-VSS) -> GND
- LED56 pad 1: Net-(LED56-VDD) -> +5V
- LED56 pad 4: Net-(LED39-VSS) -> GND
- LED57 pad 1: Net-(LED57-VDD) -> +5V
- LED57 pad 4: Net-(LED40-VSS) -> GND
- LED58 pad 1: Net-(LED58-VDD) -> +5V
- LED58 pad 4: Net-(LED41-VSS) -> GND
- LED59 pad 1: Net-(LED59-VDD) -> +5V
- LED59 pad 4: Net-(LED42-VSS) -> GND
- LED6 pad 1: +5V_LED -> +5V
- LED60 pad 1: Net-(LED60-VDD) -> +5V
- LED60 pad 4: Net-(LED43-VSS) -> GND
- LED61 pad 1: Net-(LED61-VDD) -> +5V
- LED61 pad 4: Net-(LED44-VSS) -> GND
- LED62 pad 1: Net-(LED62-VDD) -> +5V
- LED62 pad 4: Net-(LED45-VSS) -> GND
- LED63 pad 1: +5V_LED -> +5V
- LED64 pad 1: +5V_LED -> +5V
- LED65 pad 1: Net-(LED52-VDD) -> +5V
- LED66 pad 1: Net-(LED53-VDD) -> +5V
- LED67 pad 1: Net-(LED54-VDD) -> +5V
- LED68 pad 1: Net-(LED55-VDD) -> +5V
- LED69 pad 1: Net-(LED56-VDD) -> +5V
- LED7 pad 1: +5V_LED -> +5V
- LED70 pad 1: Net-(LED57-VDD) -> +5V
- LED71 pad 1: Net-(LED58-VDD) -> +5V
- LED72 pad 1: Net-(LED59-VDD) -> +5V
- LED73 pad 1: Net-(LED60-VDD) -> +5V
- LED74 pad 1: Net-(LED61-VDD) -> +5V
- LED75 pad 1: Net-(LED62-VDD) -> +5V
- LED76 pad 1: +5V_LED -> +5V
- LED77 pad 1: +5V_LED -> +5V
- LED78 pad 1: +5V_LED -> +5V
- LED79 pad 1: +5V_LED -> +5V
- LED8 pad 1: +5V_LED -> +5V
- LED80 pad 1: +5V_LED -> +5V
- LED81 pad 1: +5V_LED -> +5V
- LED82 pad 1: +5V_LED -> +5V
- LED83 pad 1: +5V_LED -> +5V
- LED84 pad 1: +5V_LED -> +5V
- LED85 pad 1: +5V_LED -> +5V
- LED86 pad 1: +5V_LED -> +5V
- LED87 pad 1: +5V_LED -> +5V
- LED9 pad 1: +5V_LED -> +5V
- U1 pad 11: /COL8 -> /COL5
- U1 pad 13: /EC11_A -> /EC11_B
- U1 pad 14: /EC11_B -> Net-(U1-D7_RX)
- U1 pad 22: /COL5 -> /COL8
- U1 pad 23: Net-(U1-D17_SCK1) -> /EC11_A
- U1 pad 29: Net-(J2-MountPin) -> GND
- U1 pad 34: /LED_ENABLE -> /5V_ENABLE
- U1 pad 35: /I2C_SCL -> /I2C_SDA
- U1 pad 36: /I2C_SDA -> /I2C_SCL
- U2 pad 1: Net-(U1-D17_SCK1) -> Net-(U1-D7_RX)
- U2 pad 2: Net-(U1-D17_SCK1) -> Net-(U1-D7_RX)
- U3 pad 1: Net-(U3-SW) -> /VBAT
- U3 pad 2: GND -> Net-(U3-EP)
- U3 pad 3: unconnected-(U3-NC-Pad3) -> +5V_USB
- U3 pad 4: Net-(D89-A) -> Net-(U3-OUT)
- U3 pad 5: unconnected-(U3-NC-Pad5) -> Net-(U3-EP)
Routing:
- net GND: track 0.00 -> 2426.8 mm, vias 0 -> 21
- net +5V: track 0.00 -> 2274.8 mm, vias 0 -> 8
- net /ROW10: track 0.00 -> 454.6 mm, vias 0 -> 4
- net /COL5: track 0.00 -> 442.6 mm, vias 0 -> 11
- net /ROW6: track 0.00 -> 421.1 mm, vias 0 -> 8
- net /COL7: track 34.5 -> 448.4 mm, vias 0 -> 4
- net /COL4: track 0.00 -> 413.3 mm, vias 0 -> 10
- net /ROW11: track 0.00 -> 412.7 mm, vias 0 -> 10
- net /ROW4: track 0.00 -> 388.7 mm, vias 0 -> 4
- net /ROW2: track 0.00 -> 385.6 mm, vias 0 -> 2
- net +3V3: track 0.00 -> 376.3 mm, vias 0 -> 6
- net /EC11_B: track 0.00 -> 371.7 mm, vias 0 -> 4
- net /COL6: track 0.00 -> 370.2 mm, vias 0 -> 7
- net /ROW9: track 0.00 -> 369.1 mm, vias 0 -> 6
- net /EC11_A: track 0.00 -> 367.6 mm, vias 0 -> 4
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