File: PCB/guilty-pad-xx-accent-core-plus-yuri.kicad_sch (KiCad schematic)
At the start: 278 parts, among them J1 Conn_01x04_Socket, Q1 G1NP02ELL, SW1 SW_Push, SW10 SW_Push, SW11 SW_Push, SW12 SW_Push, SW13 SW_Push, SW14 SW_Push, SW15 SW_Push, SW16 SW_Push, SW17 SW_Push, SW18 SW_Push, SW19 SW_Push, SW2 SW_Push, SW20 SW_Push, SW21 SW_Push, SW22 SW_Push, SW23 SW_Push, SW24 SW_Push, SW25 SW_Push, SW26 SW_Push, SW27 SW_Push, SW28 SW_Push, SW29 SW_Push, SW3 SW_Push, SW30 SW_Push, SW31 SW_Push, SW32 SW_Push, SW33 SW_Push, SW34 SW_Push, SW35 SW_Push, SW36 SW_Push, SW37 SW_Push, SW38 SW_Push, SW39 SW_Push, SW4 SW_Push, SW40 SW_Push, SW41 SW_Push, SW42 SW_Push, SW43 SW_Push, SW44 SW_Push, SW45 SW_Push, SW46 SW_Push, SW47 SW_Push, SW48 SW_Push, SW49 SW_Push, SW5 SW_Push, SW50 SW_Push, SW51 SW_Push, SW52 SW_Push, SW53 SW_Push, SW54 SW_Push, SW55 SW_Push, SW56 SW_Push, SW57 SW_Push, SW58 SW_Push, SW59 SW_Push, SW6 SW_Push, SW60 SW_Push, SW61 SW_Push, SW62 SW_Push, SW63 SW_Push, SW64 SW_Push, SW65 SW_Push, SW66 SW_Push, SW67 SW_Push, SW68 SW_Push, SW69 SW_Push, SW7 SW_Push, SW70 SW_Push, SW71 SW_Push, SW72 SW_Push, SW73 SW_Push, SW74 SW_Push, SW75 SW_Push, SW76 SW_Push, SW77 SW_Push, SW78 SW_Push, SW79 SW_Push, SW8 SW_Push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

Commit message: idkkkkkkk
Parts:
- removed Q1: G1NP02ELL, Package_TO_SOT_SMD:TSOT-23-6_HandSoldering, symbol ggxxacpy:G1NP02ELL
- removed U1: XIAO-nRF52840-SMD, OPL:XIAO-nRF52840-SMD, symbol Seeed_Studio_XIAO_Series:XIAO-nRF52840-SMD
- removed U4: AW9523B, Package_DFN_QFN:QFN-24-1EP_4x4mm_P0.5mm_EP2.7x2.7mm, symbol Interface_Expansion:AW9523B
- added C10: 4.7uF, Capacitor_SMD:C_0201_0603Metric, symbol KiCad:C_Small
- added C20: 22uF, Capacitor_SMD:C_0201_0603Metric, symbol Device:C
- added C22: 1uF, Capacitor_SMD:C_0201_0603Metric, symbol Device:C_Small
- added D90, D91: D, Diode_SMD:D_SOD-323_HandSoldering, symbol Device:D
- added D92: D, symbol Device:D
- added D93, D94: D, Diode_SMD:D_0201_0603Metric, symbol Device:D
- added D95, D96: D, Diode_SMD:D_SOD-323, symbol Device:D
- added L2: 2.2uH, Inductor_SMD:L_0201_0603Metric, symbol Device:L_Small
- added Q1, Q3: Q_PMOS, Package_TO_SOT_SMD:SOT-23_Handsoldering, symbol Device:Q_PMOS
- added Q2: Q_PMOS, guilty-devboard-idk:Vishay_PowerPAK_SC70-6L_Single, symbol Device:Q_PMOS
- added R13, R18: 1M, Resistor_SMD:R_0201_0603Metric, symbol Device:R_Small
- added R5: 4.7kΩ, Capacitor_SMD:C_0402_1005Metric_Pad0.74x0.62mm_HandSolder, symbol Device:R
- added R6: 2.2k, symbol Device:R
- added TP3, TP4: TestPoint, TestPoint:TestPoint_Pad_D1.5mm, symbol Connector:TestPoint
- added U4: PCA9555PW, Package_SO:TSSOP-24_4.4x7.8mm_P0.65mm, symbol Interface_Expansion:PCA9555PW
- added U5: 74LV1T08GW, Package_TO_SOT_SMD:SOT-353_SC-70-5, symbol 74xx:74LV1T08GW
- added U6: TP4056, Package_SO:SOP-8-1EP_4.57x4.57mm_P1.27mm_EP4.57x4.45mm, symbol PCM_marbastlib-various:TP4056
- added U7: LD1117S33TR_SOT223, Package_TO_SOT_SMD:SOT-223-3_TabPin2, symbol Regulator_Linear:LD1117S33TR_SOT223
- added U8: MIC2876-5.0YMT-TR, easyeda2kicad:UDFN-8_L2.0-W2.0-P0.50-BL-EP, symbol easyeda2kicad:MIC2876-5.0YMT-TR
- D1, D10, D11, D12, D13, D14, D15, D16, D17, D18, D19, D2, D20, D21, D22, D23, D24, D25, D26, D27, D28, D29, D3, D30, D31, D32, D33, D34, D35, D36, D37, D38, D39, D4, D40, D41, D42, D43, D44, D45, D46, D47, D48, D49, D5, D50, D51, D52, D53, D54, D55, D56, D57, D58, D59, D6, D60, D61, D62, D63, D64, D65, D66, D67, D68, D69, D7, D70, D71, D72, D73, D74, D75, D76, D77, D78, D79, D8, D80, D81, D82, D83, D84, D85, D86, D87, D9: footprint Diode_SMD:D_SMA_Handsoldering -> (none)
- D88, D89: footprint Diode_SMD:D_SMA_Handsoldering -> Diode_SMD:D_SOD-323_HandSoldering
- LED1, LED10, LED11, LED12, LED13, LED14, LED15, LED16, LED17, LED18, LED19, LED2, LED20, LED21, LED22, LED23, LED24, LED25, LED26, LED27, LED28, LED29, LED3, LED30, LED31, LED32, LED33, LED34, LED35, LED36, LED37, LED38, LED39, LED4, LED40, LED41, LED42, LED43, LED44, LED45, LED46, LED47, LED48, LED49, LED5, LED50, LED51, LED52, LED53, LED54, LED55, LED56, LED57, LED58, LED59, LED6, LED60, LED61, LED62, LED63, LED64, LED65, LED66, LED67, LED68, LED69, LED7, LED70, LED71, LED72, LED73, LED74, LED75, LED76, LED77, LED78, LED79, LED8, LED80, LED81, LED82, LED83, LED84, LED85, LED86, LED87, LED9: value MX_SK6803MINI-E -> SK6803MINI-E; symbol ggxxacpy:MX_SK6803MINI-E -> ggxxacpy:SK6803MINI-E
- SW1, SW10, SW11, SW12, SW13, SW14, SW15, SW16, SW17, SW18, SW19, SW2, SW20, SW21, SW22, SW23, SW24, SW25, SW26, SW27, SW28, SW3, SW30, SW31, SW32, SW33, SW35, SW36, SW37, SW38, SW39, SW4, SW40, SW41, SW42, SW43, SW44, SW45, SW46, SW48, SW49, SW5, SW50, SW52, SW53, SW54, SW55, SW56, SW57, SW58, SW59, SW6, SW60, SW61, SW62, SW65, SW66, SW67, SW68, SW69, SW7, SW70, SW71, SW72, SW73, SW74, SW76, SW8, SW85, SW86, SW87, SW9: footprint gpxxacpy:SW_Cherry_MX_1.00u_PCB -> (none)
- SW29: footprint gpxxacpy:SW_Cherry_MX_2.00u_PCB -> (none)
- SW34, SW47: footprint gpxxacpy:SW_Cherry_MX_1.50u_PCB -> (none)
- SW51: footprint gpxxacpy:SW_Cherry_MX_1.75u_PCB -> (none)
- SW63, SW64: footprint gpxxacpy:SW_Cherry_MX_2.25u_PCB -> (none)
- SW75: footprint gpxxacpy:SW_Cherry_MX_2.75u_PCB -> (none)
- SW77, SW78, SW79, SW81, SW82, SW83, SW84: footprint gpxxacpy:SW_Cherry_MX_1.25u_PCB -> (none)
- SW80: footprint gpxxacpy:SW_Cherry_MX_6.25u_PCB -> (none)
- renumbered SW88 to SW89
Connections:
- net LED_GND is gone; now on net GND: C2.1, LED1.4 (VSS), LED10.4 (VSS), LED11.4 (VSS), LED12.4 (VSS), LED13.4 (VSS), LED14.4 (VSS), LED15.4 (VSS), LED16.4 (VSS), LED17.4 (VSS), LED18.4 (VSS), LED19.4 (VSS)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
- net +3V3: now also R13.2, R5.1, U4.24 (VDD)
- net +5V: now also D88.1 (K), D95.1 (K), D96.1 (K), Q3.D, U5.5 (VCC); no longer D1.1 (K), LED1.1 (VDD), LED10.1 (VDD), LED11.1 (VDD), LED12.1 (VDD), LED13.1 (VDD), LED14.1 (VDD), LED15.1 (VDD), LED16.1 (VDD), LED17.1 (VDD), LED18.1 (VDD), LED19.1 (VDD)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
- net +5V_USB: now also D88.2 (A), D91.2 (A), Q1.G, U6.4 (VCC); no longer D1.2 (A)
- net COL0: now also SW1.1, SW17.1, SW34.1, SW51.1, SW64.1, SW77.1, U4.14 (IO1_1); no longer SW82.1, SW83.1, SW84.1, SW85.1, SW86.1, SW87.1
- net COL1: now also SW18.1, SW35.1, SW52.1, SW65.1, U4.15 (IO1_2); no longer SW73.1, SW74.1, SW75.1, SW76.1, SW77.1, SW79.1, SW80.1, SW81.1
- net COL2: now also SW19.1, SW2.1, SW36.1, SW53.1, SW79.1, U4.16 (IO1_3); no longer SW64.1, SW65.1, SW67.1, SW68.1, SW69.1, SW70.1, SW71.1, SW72.1
- net COL3: now also SW20.1, SW3.1, SW37.1, SW54.1, SW67.1, U4.17 (IO1_4); no longer SW55.1, SW56.1, SW57.1, SW58.1, SW59.1, SW60.1, SW61.1, SW62.1, SW63.1
- net COL4: now also SW21.1, SW38.1, SW4.1, SW55.1, SW68.1, U4.18 (IO1_5); no longer SW46.1, SW47.1, SW48.1, SW49.1, SW50.1, SW51.1, SW52.1, SW53.1, SW54.1
- net COL5: now also SW22.1, SW5.1, SW56.1, SW69.1, SW80.1, U4.19 (IO1_6); no longer SW37.1, SW38.1, SW40.1, SW41.1, SW42.1, SW43.1, SW44.1, SW45.1
- net COL6: now also SW23.1, SW40.1, SW57.1, SW6.1, SW70.1, U4.20 (IO1_7); no longer SW28.1, SW29.1, SW30.1, SW31.1, SW32.1, SW33.1, SW34.1, SW35.1, SW36.1
- net COL7: now also SW41.1, SW58.1, SW7.1, SW71.1; no longer SW19.1, SW20.1, SW21.1, SW22.1, SW23.1, SW25.1, SW26.1, SW27.1
- net COL8: now also SW25.1, SW42.1, SW59.1, SW72.1, SW8.1; no longer SW10.1, SW11.1, SW12.1, SW13.1, SW14.1, SW15.1, SW16.1, SW17.1, SW18.1
- net COL9: no longer SW1.1, SW2.1, SW3.1, SW4.1, SW5.1, SW6.1, SW7.1, SW8.1, SW9.1
- net EC11_SW: no longer SW89.S1
- net GND: now also U3.2 (GND), C10.1, C20.1, C22.1, R6.2, U4.12 (VSS), U4.2 (A1), U4.21 (A0), U4.3 (A2), U5.3 (GND), U6.1 (TEMP), U6.3 (GND)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; no longer SW89.S2
- net I2C_SCL: now also U4.22 (SCL)
- net I2C_SDA: now also U4.23 (SDA)
- net LED_ENABLE: now also D90.2 (A)
- net ROW0: now also D1.1 (K), D10.1 (K), D11.1 (K), D12.1 (K), D13.1 (K), D14.1 (K), D15.1 (K), D16.1 (K), D3.1 (K), D4.1 (K), D5.1 (K), D6.1 (K)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; no longer D18.1 (K), D20.1 (K), D35.1 (K), D38.1 (K), D52.1 (K), D56.1 (K), D65.1 (K), D78.1 (K)
- net ROW1: now also D17.1 (K), D18.1 (K), D20.1 (K), D22.1 (K), D23.1 (K), D24.1 (K), D25.1 (K), D26.1 (K), D27.1 (K), D28.1 (K), D29.1 (K), D30.1 (K)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; no longer D3.1 (K), D36.1 (K), D39.1 (K), D53.1 (K), D57.1 (K), D66.1 (K), D79.1 (K)
- net ROW2: now also D34.1 (K), D35.1 (K), D36.1 (K), D37.1 (K), D38.1 (K), D39.1 (K), D40.1 (K), D41.1 (K), D42.1 (K), D43.1 (K), D44.1 (K), D46.1 (K)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; no longer D17.1 (K), D22.1 (K), D29.1 (K), D4.1 (K), D62.1 (K), D73.1 (K), D74.1 (K), D84.1 (K)
- net ROW3: now also D51.1 (K), D52.1 (K), D53.1 (K), D54.1 (K), D55.1 (K), D56.1 (K), D57.1 (K), D58.1 (K), D59.1 (K), D60.1 (K), D61.1 (K), D62.1 (K)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; no longer D16.1 (K), D23.1 (K), D31.1 (K), D46.1 (K), D47.1 (K), D5.1 (K), D72.1 (K), D75.1 (K), D85.1 (K)
- net ROW4: now also D65.1 (K), D66.1 (K), D68.1 (K), D69.1 (K), D70.1 (K), D71.1 (K), D72.1 (K), D73.1 (K), D74.1 (K), D75.1 (K), D76.1 (K), U4.8 (IO0_4); no longer D15.1 (K), D24.1 (K), D30.1 (K), D44.1 (K), D54.1 (K), D6.1 (K), D77.1 (K), D88.1 (K)
- net ROW5: now also D77.1 (K), D78.1 (K), D79.1 (K), D81.1 (K), D82.1 (K), D83.1 (K), D84.1 (K), D85.1 (K), D86.1 (K), U4.9 (IO0_5); no longer D14.1 (K), D25.1 (K), D34.1 (K), D42.1 (K), D51.1 (K), D58.1 (K), D68.1 (K), D7.1 (K)
- net ROW6: now also U4.10 (IO0_6); no longer D13.1 (K), D26.1 (K), D33.1 (K), D43.1 (K), D50.1 (K), D59.1 (K), D69.1 (K), D8.1 (K), D81.1 (K), D86.1 (K)
- net ROW7: now also U4.11 (IO0_7); no longer D12.1 (K), D27.1 (K), D32.1 (K), D40.1 (K), D49.1 (K), D60.1 (K), D70.1 (K), D82.1 (K), D83.1 (K), D9.1 (K)
- net ROW8: now also U4.13 (IO1_0); no longer D10.1 (K), D11.1 (K), D28.1 (K), D37.1 (K), D41.1 (K), D55.1 (K), D61.1 (K), D71.1 (K), D76.1 (K)
- net VBAT: now also Q1.D, U6.5 (BAT); no longer L1.1
- net at D82.2 (A): now also SW82.2; no longer SW81.2
- net at SW22.2: now also D22.2 (A); no longer D23.2 (A)
- net at SW24.2: now also D24.2 (A); no longer D25.2 (A)
- net at SW46.2: now also D46.2 (A); no longer D47.2 (A)
- net at D48.2 (A): now also SW48.2; no longer SW47.2
- net at SW27.2: now also D27.2 (A); no longer D28.2 (A)
- net at SW55.2: now also D55.2 (A); no longer D56.2 (A)
- net at D19.2 (A): now also SW19.2; no longer SW18.2
- net at D41.2 (A): now also SW41.2; no longer SW40.2
- net at D38.2 (A): now also SW38.2; no longer SW37.2
- net at D64.2 (A): now also SW64.2; no longer SW63.2
- net at SW2.2: now also D2.2 (A); no longer D3.2 (A)
- net at SW42.2: now also D42.2 (A); no longer D43.2 (A)
- net at D69.2 (A): now also SW69.2; no longer SW68.2
- net at D58.2 (A): now also SW58.2; no longer SW57.2
- net at D85.2 (A): now also SW85.2; no longer SW84.2
- net at SW33.2: now also D33.2 (A); no longer D34.2 (A)
- net at SW29.2: now also D29.2 (A); no longer D30.2 (A)
- net at D72.2 (A): now also SW72.2; no longer SW71.2
- net at SW67.2: now also D67.2 (A); no longer D68.2 (A)
- net at D17.2 (A): now also SW17.2; no longer SW16.2
- net at D87.2 (A): now also SW87.2; no longer SW86.2
- net at D70.2 (A): now also SW70.2; no longer SW69.2
- net at SW14.2: now also D14.2 (A); no longer D15.2 (A)
- net at SW60.2: now also D60.2 (A); no longer D61.2 (A)
- net at SW13.2: now also D13.2 (A); no longer D14.2 (A)
- net at D71.2 (A): now also SW71.2; no longer SW70.2
- net at SW5.2: now also D5.2 (A); no longer D6.2 (A)
- net at SW59.2: now also D59.2 (A); no longer D60.2 (A)
- net at D73.2 (A): now also SW73.2; no longer SW72.2
- net at SW36.2: now also D36.2 (A); no longer D37.2 (A)
- net at D8.2 (A): now also SW8.2; no longer SW7.2
- net at SW66.2: now also D66.2 (A); no longer D67.2 (A)
- net at D86.2 (A): now also SW86.2; no longer SW85.2
- net at SW62.2: now also D62.2 (A); no longer D63.2 (A)
- net at SW61.2: now also D61.2 (A); no longer D62.2 (A)
- net at SW52.2: now also D52.2 (A); no longer D53.2 (A)
- net at D4.2 (A): now also SW4.2; no longer SW3.2
- net at SW9.2: now also D9.2 (A); no longer D10.2 (A)
- net at D7.2 (A): now also SW7.2; no longer SW6.2
- net at SW56.2: now also D56.2 (A); no longer D57.2 (A)
- net at D45.2 (A): now also SW45.2; no longer SW44.2
- net at SW32.2: now also D32.2 (A); no longer D33.2 (A)
- net at SW28.2: now also D28.2 (A); no longer D29.2 (A)
- net at SW34.2: now also D34.2 (A); no longer D35.2 (A)
- net at SW65.2: now also D65.2 (A); no longer D66.2 (A)
- net at SW83.2: now also D83.2 (A); no longer D84.2 (A)
- net at D81.2 (A): now also SW81.2; no longer SW80.2
- net at SW11.2: now also D11.2 (A); no longer D12.2 (A)
- net at D54.2 (A): now also SW54.2; no longer SW53.2
- net at SW51.2: now also D51.2 (A); no longer D52.2 (A)
- net at SW1.2: now also D1.2 (A); no longer D2.2 (A)
- net at D74.2 (A): now also SW74.2; no longer SW73.2
- net at SW12.2: now also D12.2 (A); no longer D13.2 (A)
- net at SW26.2: now also D26.2 (A); no longer D27.2 (A)
- net at D18.2 (A): now also SW18.2; no longer SW17.2
- net at SW50.2: now also D50.2 (A); no longer D51.2 (A)
- net at SW49.2: now also D49.2 (A); no longer D50.2 (A)
- net at D79.2 (A): now also SW79.2; no longer SW78.2
- net at SW75.2: now also D75.2 (A); no longer D76.2 (A)
- net at SW23.2: now also D23.2 (A); no longer D24.2 (A)
- net at D39.2 (A): now also SW39.2; no longer SW38.2
- net at D21.2 (A): now also SW21.2; no longer SW20.2
- net at SW10.2: now also D10.2 (A); no longer D11.2 (A)
- net at D80.2 (A): now also SW80.2; no longer SW79.2
- net at D31.2 (A): now also SW31.2; no longer SW30.2
- net at SW35.2: now also D35.2 (A); no longer D36.2 (A)
- net at SW25.2: now also D25.2 (A); no longer D26.2 (A)
- net at SW77.2: now also D77.2 (A); no longer D78.2 (A)
- net at D44.2 (A): now also SW44.2; no longer SW43.2
- net at SW76.2: now also D76.2 (A); no longer D77.2 (A)
- net at D40.2 (A): now also SW40.2; no longer SW39.2
- new net: D93.1 (K), D94.1 (K), Q2.G
- new net: C10.2, C22.2, L2.1, Q2.S, U8.3 (IN), U8.6 (EN)
- new net: L2.2, U8.1 (SW)
- new net: C20.2, D96.2 (A), U8.5 (OUTS), U8.8 (OUT)
- new net: R13.1, R18.2, U8.7 (/PG)
- new net: D68.2 (A), SW68.2
- new net: D53.2 (A), SW53.2
- new net: R6.1, U6.2 (PROG)
- new net: D84.2 (A), SW84.2
- new net: D3.2 (A), SW3.2
- new net: D37.2 (A), SW37.2
- new net: D30.2 (A), SW30.2
- new net: L1.1, Q1.S
- new net: Q3.G, U5.4 (Y)
- new net: D90.1 (K), D91.1 (K), U5.1 (B), U5.2 (A)
- new net: D43.2 (A), SW43.2
- new net: D63.2 (A), SW63.2
- new net: D15.2 (A), SW15.2
- new net: D78.2 (A), SW78.2
- new net: D57.2 (A), SW57.2
- new net: D47.2 (A), SW47.2
- new net: D6.2 (A), SW6.2
- new net: R5.2, U4.1 (~{INT})
- new net +5V_LED: LED1.1 (VDD), LED10.1 (VDD), LED11.1 (VDD), LED12.1 (VDD), LED13.1 (VDD), LED14.1 (VDD), LED15.1 (VDD), LED16.1 (VDD), LED17.1 (VDD), LED18.1 (VDD), LED19.1 (VDD), LED2.1 (VDD)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
- new net +BATT: Q2.D
- new net 5V_BOOST_ENABLE: D94.2 (A)
- new net 5V_POWER_GOOD: R18.1
- new net CHARGE_CHRG: U6.7 (CHRG)
- new net CHARGE_ENABLE: U6.8 (CE)
- new net CHARGE_STDBY: U6.6 (STDBY)
- new net EC11_SW1: D92.2 (A), SW89.S1, SW89.S2
- new net VBUS: D93.2 (A), D95.2 (A)
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Other:
- added sheet Switches (leds.kicad_sch)
- note added: "5V power circuitry"
- note added: "AGND would be AGND (connected to GND at *one* point) but this is the only thing using AGND so just connecting it to GND directly"
- note added: "capacitors should be as close as possible"
- note added: "connect /PG to AGND if unused"
- note added: "connector for batt, voltage divider, charging"
- note added: "could use EN pin to enable/disable, but only accepts up to VIN, and if on USB, then VBUS is applied, and VBUS > VIN so to make it work would require running USB through it, which would be more complex and more inefficient to make it work at all would take more components than it saves"
- note added: "hypothetically, if the battery and usb were both hooked up while discharging, then current would *probably* be split between the two sources and work fine. this would *probably* be fine with diodes there (on boost converter VOUT and xiao's +5V_USB), but we can't do that, as we have to account for battery charging over the same VBAT line because of this, there is a MOSFET that switches the boost c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"
- note added: "note 4.8A switching current != 4.8A output current absolute theoretical max ~2.5A output current this diode is only rated for 2A and i only guarantee 1A based off datahseet"
- note added: "note to self: capacitor can go either here or on +LED_5V"
- note added: "recommended 4.7+ uF ^^^ capacitor here as close as possible to inductor and connected to PGND, but not required"
- note removed: "It's all 5V, but got a diode on here to 100% make sure nothing breaks in the little time between USB being connected and the boost converter turning off"
- note removed: "connector for batt & voltage divider"
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
Commit message: cleanup and add xrd to schematic, route LED data zigzag-y
Parts:
- removed R3, R4: 4.7kΩ, Capacitor_SMD:C_0402_1005Metric_Pad0.74x0.62mm_HandSolder, symbol Device:R
- removed R6: 2.2k, symbol Device:R
- removed U6: TP4056, Package_SO:SOP-8-1EP_4.57x4.57mm_P1.27mm_EP4.57x4.45mm, symbol PCM_marbastlib-various:TP4056
- removed U7: LD1117S33TR_SOT223, Package_TO_SOT_SMD:SOT-223-3_TabPin2, symbol Regulator_Linear:LD1117S33TR_SOT223
- added TP5: TestPoint, symbol Connector:TestPoint
- added U1: Guilty Devboard Xrd, symbol xrd-lib:Guilty Devboard Xrd
- TP3, TP4: footprint TestPoint:TestPoint_Pad_D1.5mm -> (none)
Connections:
- net ROW5 is gone; now on net COL17: D77.1 (K), D78.1 (K), D79.1 (K), D80.1 (K), D81.1 (K), D82.1 (K), D83.1 (K), D84.1 (K), D85.1 (K), D86.1 (K), D87.1 (K), U4.9 (IO0_5)
- net +3V3: now also U1.10 (3V3)
- net +5V_USB: now also U1.8 (5V)
- net COL8: now also SW81.1
- net COL9: now also SW26.1, SW43.1, SW60.1, SW73.1, SW82.1, SW9.1
- net GND: now also U1.25 (BAT-), U1.29 (GND), U1.9 (GND)
- net VBAT: now also U1.24 (BAT+)
- net at TP3.1: now also U1.28 (RST)
- net at LED39.2 (DOUT): now also LED38.3 (DIN); no longer LED40.3 (DIN)
- net at LED38.2 (DOUT): now also LED37.3 (DIN); no longer LED39.3 (DIN)
- net at TP4.1: now also U1.27 (CLK)
- net COL10: now reaches SW27.1
- net COL10: now also SW10.1, SW44.1, SW61.1, SW74.1, SW83.1
- net COL15: now reaches SW31.1
- net COL15: now also SW14.1, SW48.1, SW85.1
- net at LED29.3 (DIN): now also LED30.2 (DOUT); no longer LED28.2 (DOUT)
- net at LED27.2 (DOUT): now also LED26.3 (DIN); no longer LED28.3 (DIN)
- net COL11: now reaches SW28.1
- net COL11: now also SW11.1, SW45.1, SW62.1, SW75.1, SW84.1
- net at LED77.2 (DOUT): now also LED76.3 (DIN); no longer LED78.3 (DIN)
- net at LED76.2 (DOUT): now also LED75.3 (DIN); no longer LED77.3 (DIN)
- net at LED26.2 (DOUT): now also LED25.3 (DIN); no longer LED27.3 (DIN)
- net at LED81.2 (DOUT): now also LED80.3 (DIN); no longer LED82.3 (DIN)
- net at LED80.2 (DOUT): now also LED79.3 (DIN); no longer LED81.3 (DIN)
- net at LED44.3 (DIN): now also LED45.2 (DOUT); no longer LED43.2 (DOUT)
- net at LED43.3 (DIN): now also LED44.2 (DOUT); no longer LED42.2 (DOUT)
- net at LED24.2 (DOUT): now also LED48.3 (DIN); no longer LED25.3 (DIN)
- net at LED46.2 (DOUT): now also LED45.3 (DIN); no longer LED47.3 (DIN)
- net at LED46.3 (DIN): now also LED47.2 (DOUT); no longer LED45.2 (DOUT)
- net at LED34.2 (DOUT): now also LED33.3 (DIN); no longer LED35.3 (DIN)
- net at LED34.3 (DIN): now also LED35.2 (DOUT); no longer LED33.2 (DOUT)
- net at LED84.2 (DOUT): now also LED83.3 (DIN); no longer LED85.3 (DIN)
- net at LED84.3 (DIN): now also LED85.2 (DOUT); no longer LED83.2 (DOUT)
- net at LED42.3 (DIN): now also LED43.2 (DOUT); no longer LED41.2 (DOUT)
- net COL13: now reaches SW46.1
- net COL13: now also SW12.1, SW29.1, SW63.1
- net COL14: now reaches SW13.1
- net COL14: now also SW30.1, SW47.1
- net at LED75.2 (DOUT): now also LED74.3 (DIN); no longer LED76.3 (DIN)
- net at LED74.2 (DOUT): now also LED73.3 (DIN); no longer LED75.3 (DIN)
- net at LED37.2 (DOUT): now also LED36.3 (DIN); no longer LED38.3 (DIN)
- net at LED36.2 (DOUT): now also LED35.3 (DIN); no longer LED37.3 (DIN)
- net COL16: now reaches SW49.1
- net COL16: now also SW15.1, SW32.1, SW76.1, SW86.1
- net at LED87.3 (DIN): now also LED72.2 (DOUT); no longer LED86.2 (DOUT)
- net at LED86.3 (DIN): now also LED87.2 (DOUT); no longer LED85.2 (DOUT)
- net at LED25.2 (DOUT): now also LED49.3 (DIN); no longer LED26.3 (DIN)
- net at LED79.2 (DOUT): now also LED78.3 (DIN); no longer LED80.3 (DIN)
- net at LED31.3 (DIN): now also LED32.2 (DOUT); no longer LED30.2 (DOUT)
- net at LED30.3 (DIN): now also LED31.2 (DOUT); no longer LED29.2 (DOUT)
- net at LED82.2 (DOUT): now also LED81.3 (DIN); no longer LED83.3 (DIN)
- net at LED48.2 (DOUT): now also LED47.3 (DIN); no longer LED49.3 (DIN)
- net at LED41.3 (DIN): now also LED42.2 (DOUT); no longer LED40.2 (DOUT)
- net at LED73.2 (DOUT): no longer LED74.3 (DIN)
- net at LED32.3 (DIN): now also LED33.2 (DOUT); no longer LED31.2 (DOUT)
- net COL17: now reaches SW16.1
- net COL17: now also SW33.1, SW50.1, SW87.1, SW89.S1
- net at LED78.2 (DOUT): now also LED77.3 (DIN); no longer LED79.3 (DIN)
- net EC11_SW1 renamed EC11_SW2
- net EC11_SW2: no longer SW89.S1
- new net: LED27.3 (DIN), LED28.2 (DOUT)
- new net: LED85.3 (DIN), LED86.2 (DOUT)
- new net: LED40.3 (DIN), LED41.2 (DOUT)
- new net: LED28.3 (DIN), LED29.2 (DOUT)
- new net: TP5.1, U1.26 (DIO)
- new net: LED82.3 (DIN), LED83.2 (DOUT)
- new net: LED39.3 (DIN), LED40.2 (DOUT)
Other:
- removed sheet LEDs
- removed sheet Switches
- note added: "5V on batt"
- note removed: "5V power circuitry"
- moved on the sheet: C10, C20, C22, D1, D10, D11, D12, D13, D14, D15, D16, D17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

Commit message: progress idk. western duplex matrix. stuff.
Parts:
- removed C10: 4.7uF, Capacitor_SMD:C_0201_0603Metric, symbol KiCad:C_Small
- removed C20: 22uF, Capacitor_SMD:C_0201_0603Metric, symbol Device:C
- removed C22: 1uF, Capacitor_SMD:C_0201_0603Metric, symbol Device:C_Small
- removed D93, D94: D, Diode_SMD:D_0201_0603Metric, symbol Device:D
- removed D95, D96: D, Diode_SMD:D_SOD-323, symbol Device:D
- removed L2: 2.2uH, Inductor_SMD:L_0201_0603Metric, symbol Device:L_Small
- removed Q1, Q3: Q_PMOS, Package_TO_SOT_SMD:SOT-23_Handsoldering, symbol Device:Q_PMOS
- removed Q2: Q_PMOS, guilty-devboard-idk:Vishay_PowerPAK_SC70-6L_Single, symbol Device:Q_PMOS
- removed R1: 806k, Resistor_SMD:R_0402_1005Metric_Pad0.72x0.64mm_HandSolder, symbol Device:R
- removed R13, R18: 1M, Resistor_SMD:R_0201_0603Metric, symbol Device:R_Small
- removed R2: 2M, Resistor_SMD:R_0402_1005Metric_Pad0.72x0.64mm_HandSolder, symbol Device:R
- removed R5: 4.7kΩ, Capacitor_SMD:C_0402_1005Metric_Pad0.74x0.62mm_HandSolder, symbol Device:R
- removed TP3, TP4, TP5: TestPoint, symbol Connector:TestPoint
- removed U4: PCA9555PW, Package_SO:TSSOP-24_4.4x7.8mm_P0.65mm, symbol Interface_Expansion:PCA9555PW
- removed U5: 74LV1T08GW, Package_TO_SOT_SMD:SOT-353_SC-70-5, symbol 74xx:74LV1T08GW
- removed U8: MIC2876-5.0YMT-TR, easyeda2kicad:UDFN-8_L2.0-W2.0-P0.50-BL-EP, symbol easyeda2kicad:MIC2876-5.0YMT-TR
- added J2: Conn_01x04_MountingPin, Connector_JST:JST_SH_BM04B-SRSS-TB_1x04-1MP_P1.00mm_Vertical, symbol Connector_Generic_MountingPin:Conn_01x04_MountingPin
- added Q1: AO3401A, Package_TO_SOT_SMD:SOT-23, symbol Transistor_FET:AO3401A
- added Q2: Q_NMOS, symbol Device:Q_NMOS
- D1, D10, D11, D12, D13, D14, D15, D16, D17, D18, D19, D2, D20, D21, D22, D23, D24, D25, D26, D27, D28, D29, D3, D30, D31, D32, D33, D34, D35, D36, D37, D38, D39, D4, D40, D41, D42, D43, D44, D45, D46, D47, D48, D49, D5, D50, D51, D52, D53, D54, D55, D56, D57, D58, D59, D6, D60, D61, D62, D63, D64, D65, D66, D67, D68, D69, D7, D70, D71, D72, D73, D74, D75, D76, D77, D78, D79, D8, D80, D81, D82, D83, D84, D85, D86, D87, D9, D92: footprint (none) -> Diode_SMD:D_SOD-323_HandSoldering
- D88: footprint Diode_SMD:D_SOD-323_HandSoldering -> (none)
- SW1, SW10, SW11, SW12, SW13, SW14, SW15, SW16, SW17, SW18, SW19, SW2, SW20, SW21, SW22, SW23, SW24, SW25, SW26, SW27, SW28, SW29, SW3, SW30, SW31, SW32, SW33, SW35, SW36, SW37, SW38, SW39, SW4, SW40, SW41, SW42, SW43, SW44, SW45, SW46, SW48, SW49, SW5, SW50, SW52, SW53, SW54, SW55, SW56, SW57, SW58, SW59, SW6, SW60, SW61, SW62, SW63, SW64, SW65, SW66, SW67, SW68, SW69, SW7, SW70, SW71, SW72, SW73, SW74, SW75, SW76, SW8, SW80, SW85, SW86, SW87, SW9: footprint (none) -> marbastlib-mx:SW_MX_HS_CPG151101S11_1u
- SW34, SW47: footprint (none) -> marbastlib-mx:SW_MX_HS_CPG151101S11_1.5u
- SW51: footprint (none) -> marbastlib-mx:SW_MX_HS_CPG151101S11_1.75u
- SW77, SW78, SW79, SW81, SW82, SW83, SW84: footprint (none) -> marbastlib-mx:SW_MX_HS_CPG151101S11_1.25u
- U1: footprint (none) -> xrd-lib:Guilty Devboard Xrd - SMD
Connections:
- net COL10 is gone; now on net COL5: SW10.1, SW27.1, SW44.1, SW61.1, SW74.1, SW83.1
- net COL11 is gone; now on net COL5: SW11.1, SW28.1, SW45.1, SW62.1, SW75.1, SW84.1
- net COL13 is gone; now on net COL6: SW12.1, SW29.1, SW46.1, SW63.1
- net COL14 is gone; now on net COL6: SW13.1, SW30.1, SW47.1
- net COL15 is gone; now on net COL7: SW14.1, SW31.1, SW48.1, SW85.1
- net COL16 is gone; now on net COL7: SW15.1, SW32.1, SW49.1, SW76.1, SW86.1
- net COL9 is gone; now on net COL4: SW26.1, SW43.1, SW60.1, SW73.1, SW82.1, SW9.1
- net LED_ENABLE is gone; now on an unnamed net: D90.2 (A)
- net +5V: now also LED1.1 (VDD), LED10.1 (VDD), LED11.1 (VDD), LED12.1 (VDD), LED13.1 (VDD), LED14.1 (VDD), LED15.1 (VDD), LED16.1 (VDD), LED17.1 (VDD), LED2.1 (VDD), LED3.1 (VDD), LED33.1 (VDD)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
- net +5V_USB: now also Q1.1 (G)
- net COL0: now also SW18.1, SW35.1, SW52.1, SW65.1, SW78.1, U1.3 (A/D2)
- net COL1: now also SW19.1, SW2.1, SW20.1, SW3.1, SW36.1, SW37.1, SW53.1, SW54.1, SW66.1, SW67.1, SW79.1, U1.16 (D12); no longer SW18.1, SW35.1, SW52.1, SW65.1, SW78.1
- net COL2: now also SW21.1, SW22.1, SW38.1, SW39.1, SW4.1, SW5.1, SW55.1, SW56.1, SW68.1, SW69.1, SW80.1, U1.2 (A/D1); no longer SW19.1, SW2.1, SW36.1, SW53.1, SW66.1, SW79.1
- net COL3: now also SW23.1, SW24.1, SW40.1, SW41.1, SW57.1, SW58.1, SW6.1, SW7.1, SW70.1, SW71.1, U1.15 (D11); no longer SW20.1, SW3.1, SW37.1, SW54.1, SW67.1
- net COL4: now also SW25.1, SW42.1, SW59.1, SW72.1, SW8.1, SW81.1, U1.1 (A/D0); no longer SW21.1, SW38.1, SW4.1, SW55.1, SW68.1
- net COL5: now also U1.22 (D18_MISO1); no longer SW22.1, SW39.1, SW5.1, SW56.1, SW69.1, SW80.1
- net COL6: now also U1.21 (D19_MOSI1); no longer SW23.1, SW40.1, SW57.1, SW6.1, SW70.1
- net COL7: now also U1.12 (D9_MISO); no longer SW24.1, SW41.1, SW58.1, SW7.1, SW71.1
- net COL8: now also SW16.1, SW33.1, SW50.1, SW87.1, SW89.S1, U1.11 (D10_MOSI); no longer SW25.1, SW42.1, SW59.1, SW72.1, SW8.1, SW81.1
- net EC11_A: now also U1.13 (D8_SCK)
- net EC11_B: now also U1.14 (D7_RX)
- net GND: now also Q2.S; no longer C2.1, LED35.4 (VSS), LED36.4 (VSS), LED37.4 (VSS), LED38.4 (VSS), LED39.4 (VSS), LED40.4 (VSS), LED41.4 (VSS), LED42.4 (VSS), LED43.4 (VSS), LED44.4 (VSS), LED45.4 (VSS)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
- net I2C_SCL: now also U1.35 (D25)
- net I2C_SDA: now also U1.36 (D26)
- net ROW0: now also U1.33 (D23); no longer D11.1 (K), D13.1 (K), D15.1 (K), D3.1 (K), D5.1 (K), D7.1 (K), D9.1 (K)
- net ROW1: now also D11.1 (K), D13.1 (K), D15.1 (K), D3.1 (K), D5.1 (K), D7.1 (K), D9.1 (K), U1.32 (D22); no longer D17.1 (K), D18.1 (K), D19.1 (K), D20.1 (K), D21.1 (K), D22.1 (K), D23.1 (K), D24.1 (K), D25.1 (K), D26.1 (K), D27.1 (K), D28.1 (K)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
- net ROW2: now also D17.1 (K), D19.1 (K), D21.1 (K), D23.1 (K), D25.1 (K), D27.1 (K), D29.1 (K), D31.1 (K), D33.1 (K), U1.31 (D21); no longer D34.1 (K), D35.1 (K), D36.1 (K), D37.1 (K), D38.1 (K), D39.1 (K), D40.1 (K), D41.1 (K), D42.1 (K), D43.1 (K), D44.1 (K), D45.1 (K)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
- net ROW3: now also D18.1 (K), D20.1 (K), D22.1 (K), D24.1 (K), D26.1 (K), D28.1 (K), D30.1 (K), D32.1 (K), U1.30 (D20); no longer D51.1 (K), D52.1 (K), D53.1 (K), D54.1 (K), D55.1 (K), D56.1 (K), D57.1 (K), D58.1 (K), D59.1 (K), D60.1 (K), D61.1 (K), D62.1 (K)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
- net ROW4: now also D34.1 (K), D36.1 (K), D38.1 (K), D40.1 (K), D42.1 (K), D44.1 (K), D46.1 (K), D48.1 (K), D50.1 (K), U1.7 (D6_TX); no longer D64.1 (K), D65.1 (K), D66.1 (K), D67.1 (K), D68.1 (K), D69.1 (K), D70.1 (K), D71.1 (K), D72.1 (K), D73.1 (K), D74.1 (K), D75.1 (K)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
- net ROW6: now also D51.1 (K), D53.1 (K), D55.1 (K), D57.1 (K), D59.1 (K), D61.1 (K), D63.1 (K), D92.1 (K), U1.6 (A/D5_SCL)
- net ROW7: now also D52.1 (K), D54.1 (K), D56.1 (K), D58.1 (K), D60.1 (K), D62.1 (K), U1.19 (D15_NFC2)
- net ROW8: now also D64.1 (K), D66.1 (K), D68.1 (K), D70.1 (K), D72.1 (K), D74.1 (K), U1.5 (A/D4_SDA)
- net VBAT: now also Q1.3 (D)
- net at LED46.2 (DOUT): now also LED47.3 (DIN); no longer LED45.3 (DIN)
- net at LED46.3 (DIN): now also LED45.2 (DOUT); no longer LED47.2 (DOUT)
- net at LED55.2 (DOUT): now also LED54.3 (DIN); no longer LED56.3 (DIN)
- net at LED55.3 (DIN): now also LED56.2 (DOUT); no longer LED54.2 (DOUT)
- net at LED19.2 (DOUT): now also LED18.3 (DIN); no longer LED20.3 (DIN)
- net at LED19.3 (DIN): now also LED20.2 (DOUT); no longer LED18.2 (DOUT)
- net at LED48.2 (DOUT): now also LED49.3 (DIN); no longer LED47.3 (DIN)
- net at LED48.3 (DIN): now also LED47.2 (DOUT); no longer LED24.2 (DOUT)
- net at LED21.3 (DIN): now also LED22.2 (DOUT); no longer LED20.2 (DOUT)
- net at LED73.2 (DOUT): now also LED74.3 (DIN)
- net at LED73.3 (DIN): now also LED72.2 (DOUT); no longer LED74.2 (DOUT)
- net at LED57.3 (DIN): now also LED58.2 (DOUT); no longer LED56.2 (DOUT)
- net at LED24.3 (DIN): now also LED25.2 (DOUT); no longer LED23.2 (DOUT)
- net at LED62.2 (DOUT): now also LED61.3 (DIN); no longer LED63.3 (DIN)
- net at LED62.3 (DIN): now also LED63.2 (DOUT); no longer LED61.2 (DOUT)
- net at LED44.3 (DIN): now also LED43.2 (DOUT); no longer LED45.2 (DOUT)
- net at LED44.2 (DOUT): now also LED45.3 (DIN); no longer LED43.3 (DIN)
- net at LED76.2 (DOUT): now also LED87.3 (DIN); no longer LED75.3 (DIN)
- net at LED76.3 (DIN): now also LED75.2 (DOUT); no longer LED77.2 (DOUT)
- net at LED60.2 (DOUT): now also LED59.3 (DIN); no longer LED61.3 (DIN)
- net at LED53.2 (DOUT): now also LED52.3 (DIN); no longer LED54.3 (DIN)
- net at LED53.3 (DIN): now also LED54.2 (DOUT); no longer LED52.2 (DOUT)
- net at LED38.2 (DOUT): now also LED39.3 (DIN); no longer LED37.3 (DIN)
- net at LED38.3 (DIN): now also LED37.2 (DOUT); no longer LED39.2 (DOUT)
- net at LED34.2 (DOUT): now also LED35.3 (DIN); no longer LED33.3 (DIN)
- net at LED34.3 (DIN): now also LED17.2 (DOUT); no longer LED35.2 (DOUT)
- net at LED51.2 (DOUT): now also LED64.3 (DIN); no longer LED52.3 (DIN)
- net at LED51.3 (DIN): now also LED52.2 (DOUT); no longer LED50.2 (DOUT)
- net at LED42.3 (DIN): now also LED41.2 (DOUT); no longer LED43.2 (DOUT)
- net at LED23.3 (DIN): now also LED24.2 (DOUT); no longer LED22.2 (DOUT)
- net at U2.1 (B), U2.2 (A): now also U1.23 (D17_SCK1)
- net at L1.1: now also Q1.2 (S)
- net at LED21.2 (DOUT): now also LED20.3 (DIN); no longer LED22.3 (DIN)
- net at LED36.3 (DIN): now also LED35.2 (DOUT); no longer LED37.2 (DOUT)
- net at LED40.3 (DIN): now also LED39.2 (DOUT); no longer LED41.2 (DOUT)
- net at LED42.2 (DOUT): now also LED43.3 (DIN); no longer LED41.3 (DIN)
- net 5V_ENABLE: now reaches D90.1 (K), D91.1 (K)
- net 5V_ENABLE: now also Q2.G
- net at U1.28 (RST): now also J2.3 (Pin_3)
- net ROW11: now reaches U1.17 (D13)
- net ROW11: now also D78.1 (K), D80.1 (K), D82.1 (K), D84.1 (K), D86.1 (K)
- net ROW9: now reaches U1.18 (D14_NFC1)
- net ROW9: now also D65.1 (K), D67.1 (K), D69.1 (K), D71.1 (K), D73.1 (K), D75.1 (K), D76.1 (K)
- net ROW5: now reaches U1.20 (D16_A6)
- net ROW5: now also D49.1 (K)
- net at U1.26 (DIO): now also J2.1 (Pin_1)
- net at U1.27 (CLK): now also J2.2 (Pin_2)
- net ROW10: now reaches U1.4 (A/D3)
- net ROW10: now also D77.1 (K), D79.1 (K), D81.1 (K), D83.1 (K), D85.1 (K), D87.1 (K)
- net at LED60.3 (DIN): now also LED61.2 (DOUT); no longer LED59.2 (DOUT)
- net at LED57.2 (DOUT): now also LED56.3 (DIN); no longer LED58.3 (DIN)
- net at LED16.2 (DOUT): now also LED33.3 (DIN); no longer LED17.3 (DIN)
- net at LED36.2 (DOUT): now also LED37.3 (DIN); no longer LED35.3 (DIN)
- net at LED40.2 (DOUT): now also LED41.3 (DIN); no longer LED39.3 (DIN)
- removed net +5V_LED: LED1.1 (VDD), LED10.1 (VDD), LED11.1 (VDD), LED12.1 (VDD), LED13.1 (VDD), LED14.1 (VDD), LED15.1 (VDD), LED16.1 (VDD), LED17.1 (VDD), LED18.1 (VDD), LED19.1 (VDD), LED2.1 (VDD)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
- removed net COL17: D77.1 (K), D78.1 (K), D79.1 (K), D80.1 (K), D81.1 (K), D82.1 (K), D83.1 (K), D84.1 (K), D85.1 (K), D86.1 (K), D87.1 (K), SW16.1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
- new net: LED29.1 (VDD), LED46.1 (VDD)
- new net: LED55.1 (VDD), LED68.1 (VDD)
- new net: LED38.4 (VSS), LED55.4 (VSS)
- new net: LED19.1 (VDD), LED36.1 (VDD)
- new net: LED31.1 (VDD), LED48.1 (VDD)
- new net: LED20.1 (VDD), LED37.1 (VDD)
- new net: LED60.1 (VDD), LED73.1 (VDD)
- new net: LED56.1 (VDD), LED69.1 (VDD)
- new net: LED39.4 (VSS), LED56.4 (VSS)
- new net: LED24.1 (VDD), LED41.1 (VDD)
- new net: LED53.1 (VDD), LED66.1 (VDD)
- new net: LED62.1 (VDD), LED75.1 (VDD)
- new net: LED45.4 (VSS), LED62.4 (VSS)
- new net: LED28.1 (VDD), LED45.1 (VDD)
- new net: LED27.1 (VDD), LED44.1 (VDD)
- new net: LED44.4 (VSS), LED61.4 (VSS)
- new net: LED61.1 (VDD), LED74.1 (VDD)
- new net: LED36.4 (VSS), LED53.4 (VSS)
- new net: LED25.1 (VDD), LED42.1 (VDD)
- new net: LED32.1 (VDD), LED49.1 (VDD)
- new net: LED21.1 (VDD), LED38.1 (VDD)
- new net: LED30.1 (VDD), LED47.1 (VDD)
- new net: LED26.1 (VDD), LED43.1 (VDD)
- new net: LED43.4 (VSS), LED60.4 (VSS)
- new net: J2.4 (Pin_4), J2.MP (MountPin), U1.29 (GND)
- new net: LED50.2 (DOUT), LED63.3 (DIN)
- new net: LED23.1 (VDD), LED40.1 (VDD)
- new net: LED22.3 (DIN), LED23.2 (DOUT)
- new net: LED59.1 (VDD), LED72.1 (VDD)
- new net: LED22.1 (VDD), LED39.1 (VDD)
- new net: LED37.4 (VSS), LED54.4 (VSS)
- new net: LED41.4 (VSS), LED58.4 (VSS)
- new net: LED42.4 (VSS), LED59.4 (VSS)
- new net: LED18.1 (VDD), LED35.1 (VDD)
- new net: LED17.3 (DIN), LED18.2 (DOUT)
- new net: LED52.1 (VDD), LED65.1 (VDD)
- new net: LED58.3 (DIN), LED59.2 (DOUT)
- new net: LED74.2 (DOUT), LED75.3 (DIN)
- new net: LED58.1 (VDD), LED71.1 (VDD)
- new net: LED40.4 (VSS), LED57.4 (VSS)
- new net: LED57.1 (VDD), LED70.1 (VDD)
- new net: LED35.4 (VSS), LED52.4 (VSS)
- new net: LED54.1 (VDD), LED67.1 (VDD)
- new net 5V_GND: C2.1, Q2.D, U3.2 (GND)
Other:
- note added: "5V boost conversion"
- note added: "LED control circuitry"
- note added: "LED17"
- note added: "LED33"
- note added: "LED34"
- note added: "LED50"
- note added: "LED51"
- note added: "LED63"
- note added: "LED64"
- note added: "LED76"
- note added: "LED77"
- note added: "LED87"
- note added: "NMOS must have Vgs(th) < 3.3V (under 3V to be safe, easily available anyways)"
- note added: "devboard only supplies 5V when on USB"
- note added: "notes: - BAS16WS-BL for power diodes (C5264609)"
- note added: "western duplex matrix"
- note removed: "5V on batt"
- note removed: "AGND would be AGND (connected to GND at *one* point) but this is the only thing using AGND so just connecting it to GND directly"
- note removed: "The XIAO nrf52840 only supplies 5V when on USB"
- note removed: "boost conversion and LED control circuitry"
- note removed: "capacitors should be as close as possible"
- note removed: "connect /PG to AGND if unused"
- note removed: "could use EN pin to enable/disable, but only accepts up to VIN, and if on USB, then VBUS is applied, and VBUS > VIN so to make it work would require running USB through it, which would be more complex and more inefficient to make it work at all would take more components than it saves"
- note removed: "hypothetically, if the battery and usb were both hooked up while discharging, then current would *probably* be split between the two sources and work fine. this would *probably* be fine with diodes there (on boost converter VOUT and xiao's +5V_USB), but we can't do that, as we have to account for battery charging over the same VBAT line because of this, there is a MOSFET that switches the boost c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"
- note removed: "i2c setup"
- note removed: "note 4.8A switching current != 4.8A output current absolute theoretical max ~2.5A output current this diode is only rated for 2A and i only guarantee 1A based off datahseet"
- note removed: "note to self: capacitor can go either here or on +LED_5V"
- note removed: "recommended 4.7+ uF ^^^ capacitor here as close as possible to inductor and connected to PGND, but not required"
- moved on the sheet: C2, D1, D10, D11, D12, D13, D14, D15, D16, D17, D18, D19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

Commit message: finish schematic and routing
Parts:
- removed C2: 10μF, Capacitor_SMD:C_0603_1608Metric_Pad1.08x0.95mm_HandSolder, symbol Device:C
- removed D90, D91: D, Diode_SMD:D_SOD-323_HandSoldering, symbol Device:D
- removed L1: 15μH, Inductor_SMD_Wurth:L_Wurth_WE-LQSH-4020, symbol Device:L
- removed Q1: AO3401A, Package_TO_SOT_SMD:SOT-23, symbol Transistor_FET:AO3401A
- removed Q2: Q_NMOS, symbol Device:Q_NMOS
- removed U3: TPS613222ADBV, Package_TO_SOT_SMD:SOT-23-5, symbol Regulator_Switching:TPS613222ADBV
- added C1: 0.1uF, Capacitor_SMD:C_0603_1608Metric, symbol Device:C_Small
- added C10: 4.7uF, Capacitor_SMD:C_0603_1608Metric, symbol KiCad:C_Small
- added C20, C21, C23: 22uF, Capacitor_SMD:C_0603_1608Metric, symbol Device:C
- added C22: 1uF, Capacitor_SMD:C_0603_1608Metric, symbol Device:C_Small
- added L2: 2.2uH, Inductor_SMD:L_0805_2012Metric, symbol Device:L_Small
- added R1: 1M, Resistor_SMD:R_0603_1608Metric, symbol Device:R_Small
- added U3: SiP32408, gpxxacpy:UDFN-4-1EP_1.2x1.6mm_P0.5mm_EP0.86x0.5mm, symbol ggxxacpy:SiP32408
- added U8: MIC2876-5.0YMT-TR, easyeda2kicad:UDFN-8_L2.0-W2.0-P0.50-BL-EP, symbol easyeda2kicad:MIC2876-5.0YMT-TR
- D88: footprint (none) -> Diode_SMD:D_SOD-323_HandSoldering
Connections:
- net +5V: now also LED18.1 (VDD), LED19.1 (VDD), LED20.1 (VDD), LED21.1 (VDD), LED22.1 (VDD), LED23.1 (VDD), LED24.1 (VDD), LED25.1 (VDD), LED26.1 (VDD), LED27.1 (VDD), LED28.1 (VDD), LED29.1 (VDD), LED30.1 (VDD), LED31.1 (VDD), LED32.1 (VDD), LED35.1 (VDD), LED36.1 (VDD), LED37.1 (VDD), LED38.1 (VDD), LED39.1 (VDD), LED40.1 (VDD), LED41.1 (VDD), LED42.1 (VDD), LED43.1 (VDD), LED44.1 (VDD), LED45.1 (VDD), LED46.1 (VDD), LED47.1 (VDD), LED48.1 (VDD), LED49.1 (VDD), LED52.1 (VDD), LED53.1 (VDD), LED54.1 (VDD), LED55.1 (VDD), LED56.1 (VDD), LED57.1 (VDD), LED58.1 (VDD), LED59.1 (VDD), LED60.1 (VDD), LED61.1 (VDD), LED62.1 (VDD), LED65.1 (VDD), LED66.1 (VDD), LED67.1 (VDD), LED68.1 (VDD), LED69.1 (VDD), LED70.1 (VDD), LED71.1 (VDD), LED72.1 (VDD), LED73.1 (VDD), LED74.1 (VDD), LED75.1 (VDD), C21.2
- net +5V_USB: now also R1.2, U3.3 (EN)
- net 5V_ENABLE: now also U1.34 (D24), U8.6 (EN)
- net COL5: now also U1.11 (D10_MOSI); no longer U1.22 (D18_MISO1)
- net COL8: now also U1.22 (D18_MISO1); no longer U1.11 (D10_MOSI)
- net EC11_A: now also U1.23 (D17_SCK1); no longer U1.13 (D8_SCK)
- net EC11_B: now also U1.13 (D8_SCK); no longer U1.14 (D7_RX)
- net GND: now also J2.4 (Pin_4), J2.MP (MountPin), LED35.4 (VSS), LED36.4 (VSS), LED37.4 (VSS), LED38.4 (VSS), LED39.4 (VSS), LED40.4 (VSS), LED41.4 (VSS), LED42.4 (VSS), LED43.4 (VSS), LED44.4 (VSS), LED45.4 (VSS), LED47.4 (VSS), LED48.4 (VSS), LED49.4 (VSS), LED50.4 (VSS), LED52.4 (VSS), LED53.4 (VSS), LED54.4 (VSS), LED55.4 (VSS), LED56.4 (VSS), LED57.4 (VSS), LED58.4 (VSS), LED59.4 (VSS), LED60.4 (VSS), LED61.4 (VSS), LED62.4 (VSS), U1.29 (GND), C1.2, C10.1, C20.1, C21.1, C22.1, U8.2 (PGND), U8.4 (AGND), U8.7 (/PG), U8.9 (EP)
- net I2C_SCL: now also U1.36 (D26); no longer U1.35 (D25)
- net I2C_SDA: now also U1.35 (D25); no longer U1.36 (D26)
- net ROW5: now also D35.1 (K), D37.1 (K), D39.1 (K), D41.1 (K), D43.1 (K), D45.1 (K), D47.1 (K)
- net VBAT: now also C23.2, U3.1 (IN)
- net at U2.1 (B), U2.2 (A): now also U1.14 (D7_RX); no longer U1.23 (D17_SCK1)
- net at D89.2 (A): now also C20.2, U8.5 (OUTS), U8.8 (OUT)
- new net: C23.1, R1.1, U3.2 (GND), U3.5 (EP)
- new net: C1.1, C10.2, C22.2, L2.1, U3.4 (OUT), U8.3 (IN)
- new net: L2.2, U8.1 (SW)
- no-connect marks 0 -> 1
Other:
- note added: "connector for batt"
- note added: "protection circuit won't do too much since it *only* helps with the LEDs but figured why not, just a couple more components"
- note removed: "NMOS must have Vgs(th) < 3.3V (under 3V to be safe, easily available anyways)"
- note removed: "connector for batt, voltage divider, charging"
- moved on the sheet: D88, D89, U2

Commit message: update with fixed xrd footprint, fix oled pinout, fix some silkscreen stuff, idk what else
Connections:
- net +3V3: now also J1.2 (Pin_2); no longer J1.1 (Pin_1)
- net GND: now also J1.1 (Pin_1); no longer J1.2 (Pin_2)
- net I2C_SCL: now also J1.3 (Pin_3), U1.35 (D25); no longer J1.4 (Pin_4), U1.36 (D26)
- net I2C_SDA: now also J1.4 (Pin_4), U1.36 (D26); no longer J1.3 (Pin_3), U1.35 (D25)
